File: kicad/keyboard-with-pushbuttons-and-leds/keyboard.kicad_pcb (KiCad board)
At the start: 2 copper layers, 290 x 80 mm, 136 parts, among them J1 CONN_01X02_MALE, J2 CONN_01X02_MALE, SW1 SW_Push, SW10 SW_Push, SW11 SW_Push, SW12 SW_Push, SW13 SW_Push, SW14 SW_Push, SW15 SW_Push, SW16 SW_Push, SW17 SW_Push, SW18 SW_Push, SW19 SW_Push, SW2 SW_Push, SW20 SW_Push, SW21 SW_Push, SW22 SW_Push, SW23 SW_Push, SW24 SW_Push, SW25 SW_Push, SW26 SW_Push, SW27 SW_Push, SW28 SW_Push, SW29 SW_Push, SW3 SW_Push, SW30 SW_Push, SW31 SW_Push, SW32 SW_Push, SW33 SW_Push, SW34 SW_Push, SW35 SW_Push, SW36 SW_Push, SW37 SW_Push, SW38 SW_Push, SW39 SW_Push, SW4 SW_Push, SW40 SW_Push, SW41 SW_Push, SW42 SW_Push, SW43 SW_Push, SW44 SW_Push, SW5 SW_Push, SW6 SW_Push, SW7 SW_Push, SW8 SW_Push, SW9 SW_Push

Commit message: nearly final version of keyboard PCB
Routing:
- net GND: track 0.00 -> 213.8 mm
Changed lines of the file:
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@@
   (general
     (links 268)
-    (no_connects 47)
+    (no_connects 3)
     (area 0 90 310.000001 190.000001)
     (thickness 1.6)
     (drawings 4)
-    (tracks 485)
+    (tracks 573)
     (zones 0)
     (modules 136)
@@
   (segment (start 33.05 161.375) (end 33.675 162) (width 1) (layer B.Cu) (net 1))
   (segment (start 37.773426 164.136574) (end 53.963426 164.136574) (width 1) (layer B.Cu) (net 2))
+  (segment (start 68.25 108.038474) (end 66.503426 109.785048) (width 1) (layer B.Cu) (net 3))
+  (segment (start 66.503426 109.785048) (end 66.503426 112.175048) (width 1) (layer B.Cu) (net 3))
+  (segment (start 258.25 125.358984) (end 256.503426 127.105558) (width 1) (layer B.Cu) (net 3))
+  (segment (start 256.503426 127.105558) (end 256.503426 129.495558) (width 1) (layer B.Cu) (net 3))
+  (segment (start 238.25 125.358984) (end 236.503426 127.105558) (width 1) (layer B.Cu) (net 3))
+  (segment (start 236.503426 127.105558) (end 236.503426 129.495558) (width 1) (layer B.Cu) (net 3))
+  (segment (start 218.25 125.358984) (end 216.503426 127.105558) (width 1) (layer B.Cu) (net 3))
+  (segment (start 216.503426 127.105558) (end 216.503426 129.495558) (width 1) (layer B.Cu) (net 3))
+  (segment (start 198.25 125.358984) (end 196.503426 127.105558) (width 1) (layer B.Cu) (net 3))
+  (segment (start 196.503426 127.105558) (end 196.503426 129.495558) (width 1) (layer B.Cu) (net 3))
+  (segment (start 178.25 125.358984) (end 176.503426 127.105558) (width 1) (layer B.Cu) (net 3))
+  (segment (start 176.503426 127.105558) (end 176.503426 129.495558) (width 1) (layer B.Cu) (net 3))
+  (segment (start 188.25 108.038474) (end 186.503426 109.785048) (width 1) (layer B.Cu) (net 3))
+  (segment (start 186.503426 109.785048) (end 186.503426 112.175048) (width 1) (layer B.Cu) (net 3))
+  (segment (start 158.25 125.358984) (end 156.503426 127.105558) (width 1) (layer B.Cu) (net 3))
+  (segment (start 156.503426 127.105558) (end 156.503426 129.495558) (width 1) (layer B.Cu) (net 3))
+  (segment (start 168.25 108.038474) (end 166.503426 109.785048) (width 1) (layer B.Cu) (net 3))
+  (segment (start 166.503426 109.785048) (end 166.503426 112.175048) (width 1) (layer B.Cu) (net 3))
+  (segment (start 148.25 108.038474) (end 146.503426 109.785048) (width 1) (layer B.Cu) (net 3))
+  (segment (start 146.503426 109.785048) (end 146.503426 112.175048) (width 1) (layer B.Cu) (net 3))
+  (segment (start 138.25 125.358984) (end 136.503426 127.105558) (width 1) (layer B.Cu) (net 3))
+  (segment (start 136.503426 127.105558) (end 136.503426 129.495558) (width 1) (layer B.Cu) (net 3))
+  (segment (start 128.25 108.038474) (end 126.503426 109.785048) (width 1) (layer B.Cu) (net 3))
+  (segment (start 126.503426 109.785048) (end 126.503426 112.175048) (width 1) (layer B.Cu) (net 3))
+  (segment (start 88.25 108.038474) (end 86.503426 109.785048) (width 1) (layer B.Cu) (net 3))
+  (segment (start 86.503426 109.785048) (end 86.503426 112.175048) (width 1) (layer B.Cu) (net 3))
+  (segment (start 108.25 108.038474) (end 106.503426 109.785048) (width 1) (layer B.Cu) (net 3))
+  (segment (start 106.503426 109.785048) (end 106.503426 112.175048) (width 1) (layer B.Cu) (net 3))
+  (segment (start 118.25 125.358984) (end 116.503426 127.105558) (width 1) (layer B.Cu) (net 3))
+  (segment (start 116.503426 127.105558) (end 116.503426 129.495558) (width 1) (layer B.Cu) (net 3))
+  (segment (start 98.25 125.358984) (end 96.503426 127.105558) (width 1) (layer B.Cu) (net 3))
+  (segment (start 96.503426 127.105558) (end 96.503426 129.495558) (width 1) (layer B.Cu) (net 3))
+  (segment (start 78.25 125.358984) (end 76.503426 127.105558) (width 1) (layer B.Cu) (net 3))
+  (segment (start 76.503426 127.105558) (end 76.503426 129.495558) (width 1) (layer B.Cu) (net 3))
+  (segment (start 58.25 125.358984) (end 56.503426 127.105558) (width 1) (layer B.Cu) (net 3))
+  (segment (start 56.503426 127.105558) (end 56.503426 129.495558) (width 1) (layer B.Cu) (net 3))
+  (segment (start 38.25 125.358984) (end 36.503426 127.105558) (width 1) (layer B.Cu) (net 3))
+  (segment (start 36.503426 127.105558) (end 36.503426 129.495558) (width 1) (layer B.Cu) (net 3))
+  (segment (start 28.25 142.67949) (end 26.503426 144.426064) (width 1) (layer B.Cu) (net 3))
+  (segment (start 26.503426 144.426064) (end 26.503426 146.816064) (width 1) (layer B.Cu) (net 3))
+  (segment (start 48.25 142.67949) (end 46.503426 144.426064) (width 1) (layer B.Cu) (net 3))
+  (segment (start 46.503426 144.426064) (end 46.503426 146.816064) (width 1) (layer B.Cu) (net 3))
+  (segment (start 68.25 142.67949) (end 66.503426 144.426064) (width 1) (layer B.Cu) (net 3))
+  (segment (start 66.503426 144.426064) (end 66.503426 146.816064) (width 1) (layer B.Cu) (net 3))
+  (segment (start 88.25 142.67949) (end 86.503426 144.426064) (width 1) (layer B.Cu) (net 3))
+  (segment (start 86.503426 144.426064) (end 86.503426 146.816064) (width 1) (layer B.Cu) (net 3))
+  (segment (start 108.25 142.67949) (end 106.503426 144.426064) (width 1) (layer B.Cu) (net 3))
+  (segment (start 106.503426 144.426064) (end 106.503426 146.816064) (width 1) (layer B.Cu) (net 3))
+  (segment (start 128.25 142.67949) (end 126.503426 144.426064) (width 1) (layer B.Cu) (net 3))
+  (segment (start 126.503426 144.426064) (end 126.503426 146.816064) (width 1) (layer B.Cu) (net 3))
+  (segment (start 148.25 142.67949) (end 146.503426 144.426064) (width 1) (layer B.Cu) (net 3))
+  (segment (start 146.503426 144.426064) (end 146.503426 146.816064) (width 1) (layer B.Cu) (net 3))
+  (segment (start 168.25 142.67949) (end 166.503426 144.426064) (width 1) (layer B.Cu) (net 3))
+  (segment (start 166.503426 144.426064) (end 166.503426 146.816064) (width 1) (layer B.Cu) (net 3))
+  (segment (start 188.25 142.67949) (end 186.503426 144.426064) (width 1) (layer B.Cu) (net 3))
+  (segment (start 186.503426 144.426064) (end 186.503426 146.816064) (width 1) (layer B.Cu) (net 3))
+  (segment (start 208.25 142.67949) (end 206.503426 144.426064) (width 1) (layer B.Cu) (net 3))
+  (segment (start 206.503426 144.426064) (end 206.503426 146.816064) (width 1) (layer B.Cu) (net 3))
+  (segment (start 228.25 142.67949) (end 226.503426 144.426064) (width 1) (layer B.Cu) (net 3))
+  (segment (start 226.503426 144.426064) (end 226.503426 146.816064) (width 1) (layer B.Cu) (net 3))
+  (segment (start 248.25 142.67949) (end 246.503426 144.426064) (width 1) (layer B.Cu) (net 3))
+  (segment (start 246.503426 144.426064) (end 246.503426 146.816064) (width 1) (layer B.Cu) (net 3))
+  (segment (start 268.25 142.67949) (end 266.503426 144.426064) (width 1) (layer B.Cu) (net 3))
+  (segment (start 266.503426 144.426064) (end 266.503426 146.816064) (width 1) (layer B.Cu) (net 3))
+  (segment (start 258.25 160) (end 256.503426 161.746574) (width 1) (layer B.Cu) (net 3))
+  (segment (start 256.503426 161.746574) (end 256.503426 164.136574) (width 1) (layer B.Cu) (net 3))
+  (segment (start 238.25 160) (end 236.503426 161.746574) (width 1) (layer B.Cu) (net 3))
+  (segment (start 236.503426 161.746574) (end 236.503426 164.136574) (width 1) (layer B.Cu) (net 3))
+  (segment (start 218.25 160) (end 216.503426 161.746574) (width 1) (layer B.Cu) (net 3))
+  (segment (start 216.503426 161.746574) (end 216.503426 164.136574) (width 1) (layer B.Cu) (net 3))
+  (segment (start 198.25 160) (end 196.503426 161.746574) (width 1) (layer B.Cu) (net 3))
+  (segment (start 196.503426 161.746574) (end 196.503426 164.136574) (width 1) (layer B.Cu) (net 3))
+  (segment (start 178.25 160) (end 176.503426 161.746574) (width 1) (layer B.Cu) (net 3))
+  (segment (start 176.503426 161.746574) (end 176.503426 164.136574) (width 1) (layer B.Cu) (net 3))
+  (segment (start 158.25 160) (end 156.503426 161.746574) (width 1) (layer B.Cu) (net 3))
+  (segment (start 156.503426 161.746574) (end 156.503426 164.136574) (width 1) (layer B.Cu) (net 3))
+  (segment (start 138.25 160) (end 136.503426 161.746574) (width 1) (layer B.Cu) (net 3))
+  (segment (start 136.503426 161.746574) (end 136.503426 164.136574) (width 1) (layer B.Cu) (net 3))
+  (segment (start 118.25 160) (end 116.503426 161.746574) (width 1) (layer B.Cu) (net 3))
+  (segment (start 116.503426 161.746574) (end 116.503426 164.136574) (width 1) (layer B.Cu) (net 3))
+  (segment (start 98.25 160) (end 96.503426 161.746574) (width 1) (layer B.Cu) (net 3))
+  (segment (start 96.503426 161.746574) (end 96.503426 164.136574) (width 1) (layer B.Cu) (net 3))
+  (segment (start 78.25 160) (end 76.503426 161.746574) (width 1) (layer B.Cu) (net 3))
+  (segment (start 76.503426 161.746574) (end 76.503426 164.136574) (width 1) (layer B.Cu) (net 3))
+  (segment (start 58.25 160) (end 56.503426 161.746574) (width 1) (layer B.Cu) (net 3))
+  (segment (start 56.503426 161.746574) (end 56.503426 164.136574) (width 1) (layer B.Cu) (net 3))
+  (segment (start 38.25 160) (end 36.503426 161.746574) (width 1) (layer B.Cu) (net 3))
+  (segment (start 36.503426 161.746574) (end 36.503426 164.136574) (width 1) (layer B.Cu) (net 3))
   (segment (start 22 161) (end 19 158) (width 1) (layer B.Cu) (net 4))
   (segment (start 19 158) (end 19 125) (width 1) (layer B.Cu) (net 4))

Commit message: version of printed pcb
Parts:
- LED1, LED10, LED11, LED12, LED13, LED14, LED15, LED16, LED17, LED18, LED19, LED2, LED20, LED21, LED22, LED23, LED24, LED25, LED26, LED27, LED28, LED29, LED3, LED30, LED31, LED32, LED33, LED34, LED35, LED36, LED37, LED38, LED39, LED4, LED40, LED41, LED42, LED43, LED44, LED5, LED6, LED7, LED8, LED9: footprint WS2812B-5mm-1:LED_D5.0mm-4 -> WS2812B-5mm-1:LED_D5.0mm-4-2mm
- moved C38 20.0 mm to (64.0, 128.0)
- moved C39 20.0 mm to (84.0, 128.0)
- moved C40 20.0 mm to (104.0, 128.0)
- moved C41 20.0 mm to (124.0, 128.0)
- moved C42 20.0 mm to (144.0, 128.0)
- moved C43 20.0 mm to (164.0, 128.0)
- moved C44 20.0 mm to (184.0, 128.0)
- moved SW38 20.0 mm to (70.0, 128.0)
- moved SW39 20.0 mm to (90.0, 128.0)
- moved SW40 20.0 mm to (110.0, 128.0)
- moved SW41 20.0 mm to (130.0, 128.0)
- moved SW42 20.0 mm to (150.0, 128.0)
- moved SW43 20.0 mm to (170.0, 128.0)
- moved SW44 20.0 mm to (190.0, 128.0)
- moved C1 20.0 mm to (34.0, 180.0)
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Routing:
- net Net-(LED37-Pad2): track 223.5 -> 0.00 mm
- net Net-(LED14-Pad2): track 16.2 -> 0.00 mm
- net Net-(LED25-Pad2): track 262.7 -> 257.4 mm
- net Net-(LED12-Pad2): track 262.6 -> 257.4 mm
- net VccLed: track 1296.5 -> 1298.7 mm
- net Net-(LED24-Pad2): track 16.2 -> 14.0 mm
- net Net-(LED13-Pad2): track 16.2 -> 14.0 mm
- net Net-(LED8-Pad2): track 16.2 -> 14.0 mm
- net Net-(LED7-Pad2): track 16.2 -> 14.0 mm
- net Net-(LED6-Pad2): track 16.2 -> 14.0 mm
- net Net-(LED5-Pad2): track 16.2 -> 14.0 mm
- net Net-(LED43-Pad2): track 16.2 -> 14.0 mm
- net Net-(LED42-Pad2): track 16.2 -> 14.0 mm
- net Net-(LED41-Pad2): track 16.2 -> 14.0 mm
- net Net-(LED40-Pad2): track 16.2 -> 14.0 mm
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