File: kicad/optocouplers/optocouplers.kicad_pcb (KiCad board)
At the start: 2 copper layers, 66 parts, among them J1 Conn_02x13_Top_Bottom, Q1 PN2222A, Q2 PN2222A, Q3 PN2222A, Q4 PN2222A, Q5 PN2222A, Q6 PN2222A, Q7 PN2222A, Q8 PN2222A

Commit message: temp commit with pcb
Parts:
- added R2: 1k, Resistor_SMD:R_1206_3216Metric_Pad1.42x1.75mm_HandSolder, F.Cu at (114.5, 148.0)
- added R3: 1k, Resistor_SMD:R_1206_3216Metric_Pad1.42x1.75mm_HandSolder, F.Cu at (122.0, 147.0)
- added R4: 1k, Resistor_SMD:R_1206_3216Metric_Pad1.42x1.75mm_HandSolder, F.Cu at (127.9, 146.0)
- added R5: 1k, Resistor_SMD:R_1206_3216Metric_Pad1.42x1.75mm_HandSolder, F.Cu at (136.0, 146.0)
- added R6: 1k, Resistor_SMD:R_1206_3216Metric_Pad1.42x1.75mm_HandSolder, F.Cu at (144.0, 146.0)
- added R7: 1k, Resistor_SMD:R_1206_3216Metric_Pad1.42x1.75mm_HandSolder, F.Cu at (154.5, 146.0)
- added R8: 1k, Resistor_SMD:R_1206_3216Metric_Pad1.42x1.75mm_HandSolder, F.Cu at (161.0, 146.0)
- added R_A10: 270R, Resistor_SMD:R_1206_3216Metric_Pad1.42x1.75mm_HandSolder, F.Cu at (302.0, 89.5)
- added R_A11: 270R, Resistor_SMD:R_1206_3216Metric_Pad1.42x1.75mm_HandSolder, F.Cu at (320.0, 89.0)
- added R_A2: 270R, Resistor_SMD:R_1206_3216Metric_Pad1.42x1.75mm_HandSolder, F.Cu at (145.0, 96.0)
- added R_A3: 270R, Resistor_SMD:R_1206_3216Metric_Pad1.42x1.75mm_HandSolder, F.Cu at (159.0, 89.0)
- added R_A4: 270R, Resistor_SMD:R_1206_3216Metric_Pad1.42x1.75mm_HandSolder, F.Cu at (182.0, 89.5)
- added R_A5: 270R, Resistor_SMD:R_1206_3216Metric_Pad1.42x1.75mm_HandSolder, F.Cu at (198.0, 88.5)
- added R_A6: 270R, Resistor_SMD:R_1206_3216Metric_Pad1.42x1.75mm_HandSolder, F.Cu at (222.0, 89.0)
- added R_A7: 270R, Resistor_SMD:R_1206_3216Metric_Pad1.42x1.75mm_HandSolder, F.Cu at (241.0, 90.0)
- added R_A8: 270R, Resistor_SMD:R_1206_3216Metric_Pad1.42x1.75mm_HandSolder, F.Cu at (262.0, 91.0)
- added R_A9: 270R, Resistor_SMD:R_1206_3216Metric_Pad1.42x1.75mm_HandSolder, F.Cu at (281.0, 90.0)
- added R_B0: 270R, Resistor_SMD:R_1206_3216Metric_Pad1.42x1.75mm_HandSolder, F.Cu at (85.0, 102.0)
- added R_B10: 270R, Resistor_SMD:R_1206_3216Metric_Pad1.42x1.75mm_HandSolder, F.Cu at (286.0, 102.0)
- added R_B11: 270R, Resistor_SMD:R_1206_3216Metric_Pad1.42x1.75mm_HandSolder, F.Cu at (306.0, 103.0)
- added R_B12: 270R, Resistor_SMD:R_1206_3216Metric_Pad1.42x1.75mm_HandSolder, F.Cu at (326.0, 103.0)
- added R_B3: 270R, Resistor_SMD:R_1206_3216Metric_Pad1.42x1.75mm_HandSolder, F.Cu at (145.0, 103.0)
- added R_B4: 270R, Resistor_SMD:R_1206_3216Metric_Pad1.42x1.75mm_HandSolder, F.Cu at (166.0, 104.0)
- added R_B5: 270R, Resistor_SMD:R_1206_3216Metric_Pad1.42x1.75mm_HandSolder, F.Cu at (186.0, 103.0)
- added R_B6: 270R, Resistor_SMD:R_1206_3216Metric_Pad1.42x1.75mm_HandSolder, F.Cu at (205.0, 104.0)
- added R_B7: 270R, Resistor_SMD:R_1206_3216Metric_Pad1.42x1.75mm_HandSolder, F.Cu at (226.0, 104.0)
- added R_B8: 270R, Resistor_SMD:R_1206_3216Metric_Pad1.42x1.75mm_HandSolder, F.Cu at (247.0, 102.5)
- added R_B9: 270R, Resistor_SMD:R_1206_3216Metric_Pad1.42x1.75mm_HandSolder, F.Cu at (265.0, 103.0)
- added R_C10: 270R, Resistor_SMD:R_1206_3216Metric_Pad1.42x1.75mm_HandSolder, F.Cu at (298.0, 111.0)
- added R_C11: 270R, Resistor_SMD:R_1206_3216Metric_Pad1.42x1.75mm_HandSolder, F.Cu at (318.0, 110.0)
- added R_C2: 270R, Resistor_SMD:R_1206_3216Metric_Pad1.42x1.75mm_HandSolder, F.Cu at (137.0, 110.0)
- added R_C3: 270R, Resistor_SMD:R_1206_3216Metric_Pad1.42x1.75mm_HandSolder, F.Cu at (158.0, 111.0)
- added R_C4: 270R, Resistor_SMD:R_1206_3216Metric_Pad1.42x1.75mm_HandSolder, F.Cu at (177.0, 109.5)
- added R_C5: 270R, Resistor_SMD:R_1206_3216Metric_Pad1.42x1.75mm_HandSolder, F.Cu at (197.0, 110.0)
- added R_C6: 270R, Resistor_SMD:R_1206_3216Metric_Pad1.42x1.75mm_HandSolder, F.Cu at (217.0, 111.0)
- added R_C7: 270R, Resistor_SMD:R_1206_3216Metric_Pad1.42x1.75mm_HandSolder, F.Cu at (237.0, 110.0)
- added R_C8: 270R, Resistor_SMD:R_1206_3216Metric_Pad1.42x1.75mm_HandSolder, F.Cu at (257.0, 110.0)
- added R_C9: 270R, Resistor_SMD:R_1206_3216Metric_Pad1.42x1.75mm_HandSolder, F.Cu at (278.0, 111.0)
- added R_D10: 270R, Resistor_SMD:R_1206_3216Metric_Pad1.42x1.75mm_HandSolder, F.Cu at (310.0, 117.0)
- added R_D2: 270R, Resistor_SMD:R_1206_3216Metric_Pad1.42x1.75mm_HandSolder, F.Cu at (149.0, 117.0)
- added R_D3: 270R, Resistor_SMD:R_1206_3216Metric_Pad1.42x1.75mm_HandSolder, F.Cu at (169.0, 117.0)
- added R_D4: 270R, Resistor_SMD:R_1206_3216Metric_Pad1.42x1.75mm_HandSolder, F.Cu at (189.0, 117.0)
- added R_D5: 270R, Resistor_SMD:R_1206_3216Metric_Pad1.42x1.75mm_HandSolder, F.Cu at (209.0, 117.0)
- added R_D6: 270R, Resistor_SMD:R_1206_3216Metric_Pad1.42x1.75mm_HandSolder, F.Cu at (229.0, 117.0)
- added R_D7: 270R, Resistor_SMD:R_1206_3216Metric_Pad1.42x1.75mm_HandSolder, F.Cu at (250.0, 118.0)
- added R_D8: 270R, Resistor_SMD:R_1206_3216Metric_Pad1.42x1.75mm_HandSolder, F.Cu at (269.0, 117.0)
- added R_D9: 270R, Resistor_SMD:R_1206_3216Metric_Pad1.42x1.75mm_HandSolder, F.Cu at (289.0, 117.0)
- R1, R_A0, R_A1, R_B1, R_B2, R_C0, R_C1, R_D0, R_D1: footprint Resistors_ThroughHole:R_Axial_DIN0207_L6.3mm_D2.5mm_P10.16mm_Horizontal -> Resistor_SMD:R_1206_3216Metric_Pad1.42x1.75mm_HandSolder
- moved U_B4 70.7 mm to (164.0, 114.0)
- moved U_B5 61.6 mm to (184.0, 114.0)
- moved U_A3 57.0 mm to (160.0, 100.0)
- moved U_B6 53.8 mm to (204.0, 114.0)
- moved U_D4 53.8 mm to (188.0, 128.0)
- moved U_D10 53.3 mm to (308.0, 128.0)
- moved U_C4 50.2 mm to (176.0, 121.0)
- moved U_D5 49.9 mm to (208.0, 128.0)
- moved Q4 48.4 mm to (269.0, 175.0)
- moved Q6 48.4 mm to (267.0, 157.0)
- moved U_D9 47.0 mm to (288.0, 128.0)
- moved U_A4 46.5 mm to (180.0, 100.0)
- moved U_B7 45.8 mm to (224.0, 114.0)
- moved U_B12 44.7 mm to (324.0, 114.0)
- moved U_D6 44.0 mm to (228.0, 128.0)
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Connections:
- J1 pad 16: Net-(J1-Pad16) -> (no net)
- J1 pad 17: Net-(J1-Pad17) -> (no net)
- J1 pad 24: Net-(J1-Pad24) -> (no net)
- J1 pad 25: Net-(J1-Pad25) -> (no net)
- J1 pad 26: Net-(J1-Pad26) -> (no net)
- J1 pad 3: Net-(J1-Pad3) -> (no net)
- J1 pad 4: Net-(J1-Pad4) -> (no net)
- J1 pad 5: Net-(J1-Pad5) -> (no net)
- U_A1 pad 2: Net-(Q1-Pad3) -> Net-(Q2-Pad3)
- U_A1 pad 3: arduino_A1 -> arduino_A0
- U_A10 pad 2: Net-(Q2-Pad3) -> Net-(Q1-Pad3)
- U_A10 pad 3: arduino_A4 -> arduino_A5
- U_A2 pad 3: arduino_A2 -> arduino_A1
- U_A3 pad 2: Net-(Q1-Pad3) -> Net-(Q2-Pad3)
- U_A3 pad 3: arduino_A3 -> arduino_A1
- U_A4 pad 3: arduino_A4 -> arduino_A2
- U_A5 pad 2: Net-(Q1-Pad3) -> Net-(Q2-Pad3)
- U_A5 pad 3: arduino_A5 -> arduino_A2
- U_A6 pad 2: Net-(Q2-Pad3) -> Net-(Q1-Pad3)
- U_A6 pad 3: arduino_A0 -> arduino_A3
- U_A7 pad 3: arduino_A1 -> arduino_A3
- U_A8 pad 2: Net-(Q2-Pad3) -> Net-(Q1-Pad3)
- U_A8 pad 3: arduino_A2 -> arduino_A4
- U_A9 pad 3: arduino_A3 -> arduino_A4
- U_B0 pad 2: Net-(Q7-Pad3) -> Net-(Q3-Pad3)
- U_B1 pad 2: Net-(Q3-Pad3) -> Net-(Q4-Pad3)
- U_B10 pad 2: Net-(Q4-Pad3) -> Net-(Q3-Pad3)
- U_B10 pad 3: arduino_A3 -> arduino_A5
- U_B11 pad 3: arduino_A4 -> arduino_A5
- U_B12 pad 2: Net-(Q4-Pad3) -> Net-(Q8-Pad3)
- U_B3 pad 2: Net-(Q3-Pad3) -> Net-(Q4-Pad3)
- U_B3 pad 3: arduino_A2 -> arduino_A1
- U_B4 pad 3: arduino_A3 -> arduino_A2
- U_B5 pad 2: Net-(Q3-Pad3) -> Net-(Q4-Pad3)
- U_B5 pad 3: arduino_A4 -> arduino_A2
- U_B6 pad 3: arduino_A5 -> arduino_A3
- U_B7 pad 3: arduino_A0 -> arduino_A3
- U_B8 pad 2: Net-(Q4-Pad3) -> Net-(Q3-Pad3)
- U_B8 pad 3: arduino_A1 -> arduino_A4
- U_B9 pad 3: arduino_A2 -> arduino_A4
- U_C1 pad 2: Net-(Q5-Pad3) -> Net-(Q6-Pad3)
- U_C1 pad 3: arduino_A1 -> arduino_A0
- U_C10 pad 2: Net-(Q6-Pad3) -> Net-(Q5-Pad3)
- U_C10 pad 3: arduino_A4 -> arduino_A5
- U_C2 pad 3: arduino_A2 -> arduino_A1
- U_C3 pad 2: Net-(Q5-Pad3) -> Net-(Q6-Pad3)
- U_C3 pad 3: arduino_A3 -> arduino_A1
- U_C4 pad 3: arduino_A4 -> arduino_A2
- U_C5 pad 2: Net-(Q5-Pad3) -> Net-(Q6-Pad3)
- U_C5 pad 3: arduino_A5 -> arduino_A2
- U_C6 pad 2: Net-(Q6-Pad3) -> Net-(Q5-Pad3)
- U_C6 pad 3: arduino_A0 -> arduino_A3
- U_C7 pad 3: arduino_A1 -> arduino_A3
- U_C8 pad 2: Net-(Q6-Pad3) -> Net-(Q5-Pad3)
- U_C8 pad 3: arduino_A2 -> arduino_A4
- U_C9 pad 3: arduino_A3 -> arduino_A4
- U_D0 pad 3: arduino_A1 -> arduino_A0
- U_D1 pad 2: Net-(Q7-Pad3) -> Net-(Q8-Pad3)
- U_D1 pad 3: arduino_A2 -> arduino_A0
- U_D10 pad 2: Net-(Q8-Pad3) -> Net-(Q7-Pad3)
- U_D2 pad 3: arduino_A3 -> arduino_A1
- U_D3 pad 2: Net-(Q7-Pad3) -> Net-(Q8-Pad3)
- U_D3 pad 3: arduino_A4 -> arduino_A1
- U_D4 pad 3: arduino_A5 -> arduino_A2
- U_D5 pad 3: arduino_A0 -> arduino_A2
- U_D6 pad 2: Net-(Q8-Pad3) -> Net-(Q7-Pad3)
- U_D6 pad 3: arduino_A1 -> arduino_A3
- U_D7 pad 3: arduino_A2 -> arduino_A3
- U_D8 pad 2: Net-(Q8-Pad3) -> Net-(Q7-Pad3)
- U_D8 pad 3: arduino_A3 -> arduino_A4
Routing:
- net arduino_A0: track 28.4 -> 68.0 mm
- net arduino_A1: track 39.6 -> 0.00 mm
- net Net-(Q8-Pad3): track 0.00 -> 2.90 mm
- net Net-(Q7-Pad3): track 50.5 -> 47.6 mm

Commit message: intermediate step of optocoupler pcb
Parts:
- R1, R2, R3, R4, R5, R6, R7, R8, R_A0, R_A1, R_A10, R_A11, R_A2, R_A3, R_A4, R_A5, R_A6, R_A7, R_A8, R_A9, R_B0, R_B1, R_B10, R_B11, R_B12, R_B2, R_B3, R_B4, R_B5, R_B6, R_B7, R_B8, R_B9, R_C0, R_C1, R_C10, R_C11, R_C2, R_C3, R_C4, R_C5, R_C6, R_C7, R_C8, R_C9, R_D0, R_D1, R_D10, R_D2, R_D3, R_D4, R_D5, R_D6, R_D7, R_D8, R_D9: moved to B.Cu
- moved Q2 244.8 mm to (92.0, 100.0), turned to 90 degrees
- moved Q8 234.9 mm to (77.0, 141.0), turned to 90 degrees
- moved Q4 201.8 mm to (77.0, 113.0), turned to 90 degrees
- moved Q6 192.4 mm to (77.0, 127.0), turned to 90 degrees
- moved R8 94.3 mm to (67.0, 139.0)
- moved R7 87.5 mm to (68.0, 133.0)
- moved R6 78.6 mm to (68.0, 126.0)
- moved R5 72.7 mm to (68.5, 119.0)
- moved R4 68.5 mm to (69.0, 111.0)
- moved R3 67.6 mm to (69.0, 105.0)
- moved R2 57.5 mm to (84.5, 99.0)
- moved R_D0 29.0 mm to (109.0, 118.0)
- moved R_D1 29.0 mm to (129.0, 118.0)
- moved R_C0 23.5 mm to (96.0, 112.0), turned to 180 degrees
- moved R_C1 23.0 mm to (116.0, 112.0), turned to 180 degrees
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Routing:
- net +5V: track 0.00 -> 534.9 mm
- net Net-(Q8-Pad3): track 2.90 -> 346.4 mm
- net Net-(Q4-Pad3): track 0.00 -> 245.0 mm
- net Net-(Q2-Pad3): track 0.00 -> 244.9 mm
- net Net-(Q3-Pad3): track 29.0 -> 246.5 mm
- net Net-(Q6-Pad3): track 0.00 -> 216.2 mm
- net Net-(Q7-Pad3): track 47.6 -> 258.0 mm
- net Net-(Q5-Pad3): track 46.0 -> 244.9 mm
- net Net-(Q1-Pad3): track 30.2 -> 225.2 mm
- net arduino_A5: track 0.00 -> 129.5 mm
- net arduino_A1: track 0.00 -> 110.9 mm
- net arduino_A3: track 0.00 -> 109.7 mm
- net arduino_A4: track 0.00 -> 109.2 mm
- net arduino_A2: track 0.00 -> 108.4 mm
- net arduino_A0: track 68.0 -> 109.8 mm
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
Commit message: almost complete pcb
Parts:
- removed J1: Conn_02x13_Top_Bottom, Connectors_Multicomp:Multicomp_MC9A12-2634_2x13x2.54mm_Straight
- added Conn1: Conn_02x13_Odd_Even, Connector_Multicomp:Multicomp_MC9A12-2634_2x13_P2.54mm_Vertical, B.Cu at (104.8, 63.0)
- R1, R2, R3, R4: moved to F.Cu
- moved R_A0 100.5 mm to (41.5, 19.5)
- moved R_A1 100.5 mm to (61.5, 19.5)
- moved R_A10 100.5 mm to (243.5, 17.5)
- moved R_A11 100.5 mm to (261.5, 19.5)
- moved R_A2 100.5 mm to (81.5, 19.5)
- moved R_A3 100.5 mm to (101.5, 19.5)
- moved R_A4 100.5 mm to (121.5, 19.5)
- moved R_A5 100.5 mm to (141.5, 19.5)
- moved R_A6 100.5 mm to (161.5, 19.5)
- moved R_A7 100.5 mm to (181.5, 19.5)
- moved R_A8 100.5 mm to (201.5, 19.5)
- moved R_A9 100.5 mm to (223.5, 17.5)
- moved R_B0 100.5 mm to (25.5, 33.5)
- moved R_B1 100.5 mm to (43.5, 24.5)
- moved R_B10 100.5 mm to (223.5, 24.5)
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Routing:
- net +5V: track 534.9 -> 724.9 mm
- net arduino_A5: track 129.5 -> 268.3 mm
- net arduino_A4: track 109.2 -> 217.6 mm
- net Net-(Q8-Pad3): track 346.4 -> 242.7 mm
- net arduino_D5: track 0.00 -> 87.8 mm
- net arduino_D6: track 0.00 -> 77.2 mm
- net arduino_D7: track 0.00 -> 67.2 mm
- net arduino_A3: track 109.7 -> 175.2 mm
- net arduino_D8: track 0.00 -> 56.2 mm
- net arduino_D9: track 0.00 -> 49.2 mm
- net Net-(Q1-Pad3): track 225.2 -> 273.5 mm
- net Net-(Q2-Pad3): track 244.9 -> 290.5 mm
- net arduino_D10: track 0.00 -> 38.7 mm
- net arduino_A0: track 109.8 -> 138.1 mm
- net arduino_D11: track 0.00 -> 27.6 mm
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Other:
- board outline added: 294 x 70 mm

Commit message: Almost finished pcb
Parts:
- added REF**: 1pin, Connectors:1pin, F.Cu at (10.0, 65.0)
- added REF**: 1pin, Connectors:1pin, F.Cu at (284.0, 5.00)
- added REF**: 1pin, Connectors:1pin, F.Cu at (284.0, 65.0)
- added REF**: 1pin, Connectors:1pin, F.Cu at (10.0, 5.00)
Routing:
- added copper zone on B.Cu, net GND
- added copper zone on F.Cu, net GND

Commit message: Backup of optocouplers
Parts:
- added R_R0: 2k, Resistor_SMD:R_1206_3216Metric_Pad1.42x1.75mm_HandSolder, B.Cu at (53.0, 24.5)
- added R_R1: 2k, Resistor_SMD:R_1206_3216Metric_Pad1.42x1.75mm_HandSolder, B.Cu at (93.0, 24.5)
- added R_R2: 2k, Resistor_SMD:R_1206_3216Metric_Pad1.42x1.75mm_HandSolder, B.Cu at (133.0, 24.5)
- added R_R3: 2k, Resistor_SMD:R_1206_3216Metric_Pad1.42x1.75mm_HandSolder, B.Cu at (173.0, 24.5)
- added R_R4: 2k, Resistor_SMD:R_1206_3216Metric_Pad1.42x1.75mm_HandSolder, B.Cu at (213.0, 24.5)
- added R_R5: 2k, Resistor_SMD:R_1206_3216Metric_Pad1.42x1.75mm_HandSolder, B.Cu at (248.0, 24.5)
- Q1, Q2, Q3, Q4, Q5, Q6, Q7, Q8: footprint TO_SOT_Packages_THT:TO-92_Molded_Narrow -> Package_TO_SOT_THT:TO-92L_HandSolder
- R1, R2, R3, R4: moved to B.Cu
- moved R_B0 5.32 mm to (29.0, 29.5)
- moved R8 3.81 mm to (66.2, 63.5)
- moved R_A5 3.38 mm to (143.8, 17.0), turned to 270 degrees
- moved R_A6 3.38 mm to (163.8, 17.0), turned to 270 degrees
- moved R_A7 3.38 mm to (183.8, 17.0), turned to 270 degrees
- moved R_A8 3.38 mm to (203.8, 17.0), turned to 270 degrees
- moved R_A0 3.38 mm to (43.8, 17.0), turned to 270 degrees
- moved R_A1 3.38 mm to (63.8, 17.0), turned to 270 degrees
- moved R_A2 3.38 mm to (83.8, 17.0), turned to 270 degrees
- moved R_A3 3.38 mm to (103.8, 17.0), turned to 270 degrees
- moved R_A4 3.38 mm to (123.8, 17.0), turned to 270 degrees
- moved R_A11 3.38 mm to (263.8, 17.0), turned to 270 degrees
- moved R_C7 2.24 mm to (174.5, 32.5), turned to 180 degrees
- moved R7 1.53 mm to (59.2, 63.5)
- moved R5 1.52 mm to (45.2, 63.5)
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Connections:
- Conn1 pad 11: arduino_D9 -> arduino_D6
- Conn1 pad 13: arduino_D10 -> arduino_D7
- Conn1 pad 15: arduino_D11 -> arduino_D8
- Conn1 pad 17: arduino_D12 -> arduino_D9
- Conn1 pad 19: (no net) -> arduino_D10
- Conn1 pad 21: (no net) -> arduino_D11
- Conn1 pad 23: (no net) -> arduino_D12
- Conn1 pad 3: arduino_D5 -> (no net)
- Conn1 pad 5: arduino_D6 -> (no net)
- Conn1 pad 7: arduino_D7 -> (no net)
- Conn1 pad 9: arduino_D8 -> arduino_D5
Routing:
- net Net-(Q6-Pad3): track 216.2 -> 241.1 mm, vias 0 -> 1
- net Net-(Q8-Pad3): track 242.7 -> 258.0 mm
- net arduino_A5: track 268.3 -> 279.2 mm
- net +5V: track 724.9 -> 715.9 mm
- net arduino_D7: track 67.2 -> 59.2 mm, vias 0 -> 1
- net arduino_D6: track 77.2 -> 69.6 mm, vias 0 -> 1
- net arduino_D8: track 56.2 -> 48.5 mm, vias 0 -> 1
- net arduino_D10: track 38.7 -> 31.4 mm
- net arduino_D9: track 49.2 -> 42.0 mm
- net arduino_D5: track 87.8 -> 81.0 mm, vias 0 -> 1
- net arduino_D11: track 27.6 -> 21.2 mm
- net arduino_A2: track 134.1 -> 140.3 mm
- net arduino_A1: track 120.8 -> 126.1 mm
- net Net-(Q1-Pad3): track 273.5 -> 268.9 mm
- net Net-(Q5-Pad3): track 250.2 -> 254.0 mm
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