File: kicad/optocouplers/optocouplers.sch (KiCad schematic (older format))
At the start: 119 parts, among them Q1 PN2222A, Q2 PN2222A, Q3 PN2222A, Q4 PN2222A, Q5 PN2222A, Q6 PN2222A, Q7 PN2222A, Q8 PN2222A

Commit message: Backup of optocouplers
Parts:
- Q1, Q2, Q3, Q4, Q5, Q6, Q7, Q8: footprint Package_TO_SOT_THT:TO-92_Inline -> Package_TO_SOT_THT:TO-92L_HandSolder
Changed lines of the file:
@@
 F 0 "Q1" V 1050 4000 50  0000 L CNN
 F 1 "PN2222A" V 1300 4050 50  0000 L CNN
-F 2 "Package_TO_SOT_THT:TO-92_Inline" H 1300 4125 50  0001 L CIN
+F 2 "Package_TO_SOT_THT:TO-92L_HandSolder" H 1300 4125 50  0001 L CIN
 F 3 "" H 1100 4200 50  0001 L CNN
 	1    1100 4200
@@
 F 0 "Q2" V 2850 4000 50  0000 L CNN
 F 1 "PN2222A" V 3100 4050 50  0000 L CNN
-F 2 "Package_TO_SOT_THT:TO-92_Inline" H 3100 4125 50  0001 L CIN
+F 2 "Package_TO_SOT_THT:TO-92L_HandSolder" H 3100 4125 50  0001 L CIN
 F 3 "" H 2900 4200 50  0001 L CNN
 	1    2900 4200
@@
 F 0 "Q3" V 4650 4000 50  0000 L CNN
 F 1 "PN2222A" V 4900 4050 50  0000 L CNN
-F 2 "Package_TO_SOT_THT:TO-92_Inline" H 4900 4125 50  0001 L CIN
+F 2 "Package_TO_SOT_THT:TO-92L_HandSolder" H 4900 4125 50  0001 L CIN
 F 3 "" H 4700 4200 50  0001 L CNN
 	1    4700 4200
@@
 F 0 "Q4" V 6450 4000 50  0000 L CNN
 F 1 "PN2222A" V 6700 4050 50  0000 L CNN
-F 2 "Package_TO_SOT_THT:TO-92_Inline" H 6700 4125 50  0001 L CIN
+F 2 "Package_TO_SOT_THT:TO-92L_HandSolder" H 6700 4125 50  0001 L CIN
 F 3 "" H 6500 4200 50  0001 L CNN
 	1    6500 4200
@@
 F 0 "Q5" V 8250 4000 50  0000 L CNN
 F 1 "PN2222A" V 8500 4050 50  0000 L CNN
-F 2 "Package_TO_SOT_THT:TO-92_Inline" H 8500 4125 50  0001 L CIN
+F 2 "Package_TO_SOT_THT:TO-92L_HandSolder" H 8500 4125 50  0001 L CIN
 F 3 "" H 8300 4200 50  0001 L CNN
 	1    8300 4200
@@
 F 0 "Q6" V 10050 4000 50  0000 L CNN
 F 1 "PN2222A" V 10300 4050 50  0000 L CNN
-F 2 "Package_TO_SOT_THT:TO-92_Inline" H 10300 4125 50  0001 L CIN
+F 2 "Package_TO_SOT_THT:TO-92L_HandSolder" H 10300 4125 50  0001 L CIN
 F 3 "" H 10100 4200 50  0001 L CNN
 	1    10100 4200
@@
 F 0 "Q7" V 11850 4000 50  0000 L CNN
 F 1 "PN2222A" V 12100 4050 50  0000 L CNN
-F 2 "Package_TO_SOT_THT:TO-92_Inline" H 12100 4125 50  0001 L CIN
+F 2 "Package_TO_SOT_THT:TO-92L_HandSolder" H 12100 4125 50  0001 L CIN
 F 3 "" H 11900 4200 50  0001 L CNN
 	1    11900 4200
@@
 F 0 "Q8" V 13650 4000 50  0000 L CNN
 F 1 "PN2222A" V 13900 4050 50  0000 L CNN
-F 2 "Package_TO_SOT_THT:TO-92_Inline" H 13900 4125 50  0001 L CIN
+F 2 "Package_TO_SOT_THT:TO-92L_HandSolder" H 13900 4125 50  0001 L CIN
 F 3 "" H 13700 4200 50  0001 L CNN
 	1    13700 4200
