File: kicad/optocouplers-rewire/optocouplers.kicad_pcb (KiCad board)
At the start: 2 copper layers, 123 parts, among them Q1 PN2222A, Q2 PN2222A, Q3 PN2222A, Q4 PN2222A, Q5 PN2222A, Q6 PN2222A, Q7 PN2222A, Q8 PN2222A

Commit message: Remove paths
Routing:
- net +5V: track 460.0 -> 0.00 mm
- net Net-(Q3-Pad3): track 112.8 -> 0.00 mm
- net Net-(Q1-Pad3): track 112.8 -> 0.00 mm
- net Net-(U.A6-Pad1): track 3.45 -> 0.00 mm
- net Net-(R.D9-Pad1): track 3.45 -> 0.00 mm
- net Net-(R.D8-Pad1): track 3.45 -> 0.00 mm
- net Net-(R.D7-Pad1): track 3.45 -> 0.00 mm
- net Net-(R.D6-Pad1): track 3.45 -> 0.00 mm
- net Net-(R.D5-Pad1): track 3.45 -> 0.00 mm
- net Net-(R.D4-Pad1): track 3.45 -> 0.00 mm
- net Net-(R.D3-Pad1): track 3.45 -> 0.00 mm
- net Net-(R.D2-Pad1): track 3.45 -> 0.00 mm
- net Net-(R.D10-Pad1): track 3.45 -> 0.00 mm
- net Net-(R.D1-Pad1): track 3.45 -> 0.00 mm
- net Net-(R.D0-Pad1): track 3.45 -> 0.00 mm
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Changed lines of the file:
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@@
     )
   )
-  (segment (start 69.23 27.11) (end 69.206475 27.086475) (width 0.6) (layer "B.Cu") (net 2))
-  (segment (start 126.816475 27.086475) (end 129.23 29.5) (width 0.6) (layer "B.Cu") (net 2))
-  (segment (start 49.23 29.5) (end 49.23 27.11) (width 0.6) (layer "B.Cu") (net 2))
-  (segment (start 109.23 27.09) (end 109.233525 27.086475) (width 0.6) (layer "B.Cu") (net 2))
-  (segment (start 69.206475 27.086475) (end 89.233525 27.086475) (width 0.6) (layer "B.Cu") (net 2))
-  (segment (start 69.23 29.5) (end 69.23 27.11) (width 0.6) (layer "B.Cu") (net 2))
-  (segment (start 29.793525 27.086475) (end 49.253525 27.086475) (width 0.6) (layer "B.Cu") (net 2))
-  (segment (start 29.23 29.5) (end 29.23 27.65) (width 0.6) (layer "B.Cu") (net 2))
-  (segment (start 109.23 29.5) (end 109.23 27.09) (width 0.6) (layer "B.Cu") (net 2))
-  (segment (start 49.253525 27.086475) (end 69.206475 27.086475) (width 0.6) (layer "B.Cu") (net 2))
-  (segment (start 109.233525 27.086475) (end 126.816475 27.086475) (width 0.6) (layer "B.Cu") (net 2))
-  (segment (start 29.23 27.65) (end 29.793525 27.086475) (width 0.6) (layer "B.Cu") (net 2))
-  (segment (start 49.23 27.11) (end 49.253525 27.086475) (width 0.6) (layer "B.Cu") (net 2))
-  (segment (start 89.233525 27.086475) (end 109.233525 27.086475) (width 0.6) (layer "B.Cu") (net 2))
-  (segment (start 89.23 29.5) (end 89.23 27.09) (width 0.6) (layer "B.Cu") (net 2))
-  (segment (start 89.23 27.09) (end 89.233525 27.086475) (width 0.6) (layer "B.Cu") (net 2))
-  (segment (start 23.77 36.05) (end 263.77 36.05) (width 0.6) (layer "B.Cu") (net 4))
-  (segment (start 35.77 50.05) (end 255.77 50.05) (width 0.6) (layer "B.Cu") (net 4))
-  (segment (start 21.23 29.5) (end 21.23 27.65) (width 0.6) (layer "F.Cu") (net 22))
-  (segment (start 61.213525 27.086475) (end 81.233525 27.086475) (width 0.6) (layer "F.Cu") (net 22))
-  (segment (start 21.23 27.65) (end 21.793525 27.086475) (width 0.6) (layer "F.Cu") (net 22))
-  (segment (start 21.793525 27.086475) (end 41.206475 27.086475) (width 0.6) (layer "F.Cu") (net 22))
-  (segment (start 81.23 27.09) (end 81.233525 27.086475) (width 0.6) (layer "F.Cu") (net 22))
-  (segment (start 61.23 29.5) (end 61.23 27.10295) (width 0.6) (layer "F.Cu") (net 22))
-  (segment (start 101.23 27.16) (end 101.303525 27.086475) (width 0.6) (layer "F.Cu") (net 22))
-  (segment (start 41.23 29.5) (end 41.23 27.11) (width 0.6) (layer "F.Cu") (net 22))
-  (segment (start 61.23 27.10295) (end 61.213525 27.086475) (width 0.6) (layer "F.Cu") (net 22))
-  (segment (start 118.816475 27.086475) (end 121.23 29.5) (width 0.6) (layer "F.Cu") (net 22))
-  (segment (start 41.206475 27.086475) (end 61.213525 27.086475) (width 0.6) (layer "F.Cu") (net 22))
-  (segment (start 101.303525 27.086475) (end 118.816475 27.086475) (width 0.6) (layer "F.Cu") (net 22))
-  (segment (start 101.23 29.5) (end 101.23 27.16) (width 0.6) (layer "F.Cu") (net 22))
-  (segment (start 41.23 27.11) (end 41.206475 27.086475) (width 0.6) (layer "F.Cu") (net 22))
-  (segment (start 81.23 29.5) (end 81.23 27.09) (width 0.6) (layer "F.Cu") (net 22))
-  (segment (start 81.233525 27.086475) (end 101.303525 27.086475) (width 0.6) (layer "F.Cu") (net 22))
-  (segment (start 31.77 29.5) (end 31.77 32.95) (width 0.6) (layer "B.Cu") (net 41))
-  (segment (start 51.77 29.5) (end 51.77 32.95) (width 0.6) (layer "B.Cu") (net 42))
-  (segment (start 71.77 29.5) (end 71.77 32.95) (width 0.6) (layer "B.Cu") (net 43))
-  (segment (start 91.77 29.5) (end 91.77 32.95) (width 0.6) (layer "B.Cu") (net 44))
-  (segment (start 111.77 29.5) (end 111.77 32.95) (width 0.6) (layer "B.Cu") (net 45))
-  (segment (start 131.77 29.5) (end 131.77 32.95) (width 0.6) (layer "B.Cu") (net 46))
-  (segment (start 151.77 29.5) (end 151.77 32.95) (width 0.6) (layer "B.Cu") (net 47))
-  (segment (start 171.77 29.5) (end 171.77 32.95) (width 0.6) (layer "B.Cu") (net 48))
-  (segment (start 191.77 29.5) (end 191.77 32.95) (width 0.6) (layer "B.Cu") (net 49))
-  (segment (start 211.77 29.5) (end 211.77 32.95) (width 0.6) (layer "B.Cu") (net 50))
-  (segment (start 231.77 29.5) (end 231.77 32.95) (width 0.6) (layer "B.Cu") (net 51))
-  (segment (start 251.77 29.5) (end 251.77 32.95) (width 0.6) (layer "B.Cu") (net 52))
-  (segment (start 23.77 29.5) (end 23.77 32.95) (width 0.6) (layer "B.Cu") (net 53))
-  (segment (start 43.77 29.5) (end 43.77 32.95) (width 0.6) (layer "B.Cu") (net 54))
-  (segment (start 63.77 29.5) (end 63.77 32.95) (width 0.6) (layer "B.Cu") (net 55))
-  (segment (start 83.77 29.5) (end 83.77 32.95) (width 0.6) (layer "B.Cu") (net 56))
-  (segment (start 103.77 29.5) (end 103.77 32.95) (width 0.6) (layer "B.Cu") (net 57))
-  (segment (start 123.77 29.5) (end 123.77 32.95) (width 0.6) (layer "B.Cu") (net 58))
-  (segment (start 143.77 29.5) (end 143.77 32.95) (width 0.6) (layer "B.Cu") (net 59))
-  (segment (start 163.77 29.5) (end 163.77 32.95) (width 0.6) (layer "B.Cu") (net 60))
-  (segment (start 183.77 29.5) (end 183.77 32.95) (width 0.6) (layer "B.Cu") (net 61))
-  (segment (start 203.77 29.5) (end 203.77 32.95) (width 0.6) (layer "B.Cu") (net 62))
-  (segment (start 223.77 29.5) (end 223.77 32.95) (width 0.6) (layer "B.Cu") (net 63))
-  (segment (start 243.77 29.5) (end 243.77 32.95) (width 0.6) (layer "B.Cu") (net 64))
-  (segment (start 263.77 29.5) (end 263.77 32.95) (width 0.6) (layer "B.Cu") (net 65))
-  (segment (start 35.77 43.5) (end 35.77 46.95) (width 0.6) (layer "B.Cu") (net 66))
-  (segment (start 55.77 43.5) (end 55.77 46.95) (width 0.6) (layer "B.Cu") (net 67))
-  (segment (start 75.77 43.5) (end 75.77 46.95) (width 0.6) (layer "B.Cu") (net 68))
-  (segment (start 95.77 43.5) (end 95.77 46.95) (width 0.6) (layer "B.Cu") (net 69))
-  (segment (start 115.77 43.5) (end 115.77 46.95) (width 0.6) (layer "B.Cu") (net 70))
-  (segment (start 135.77 43.5) (end 135.77 46.95) (width 0.6) (layer "B.Cu") (net 71))
-  (segment (start 155.77 43.5) (end 155.77 46.95) (width 0.6) (layer "B.Cu") (net 72))
-  (segment (start 175.77 43.5) (end 175.77 46.95) (width 0.6) (layer "B.Cu") (net 73))
-  (segment (start 195.77 43.5) (end 195.77 46.95) (width 0.6) (layer "B.Cu") (net 74))
-  (segment (start 215.77 43.5) (end 215.77 46.95) (width 0.6) (layer "B.Cu") (net 75))
-  (segment (start 235.77 43.5) (end 235.77 46.95) (width 0.6) (layer "B.Cu") (net 76))
-  (segment (start 255.77 43.5) (end 255.77 46.95) (width 0.6) (layer "B.Cu") (net 77))
-  (segment (start 47.77 43.5) (end 47.77 46.95) (width 0.6) (layer "B.Cu") (net 78))
-  (segment (start 67.77 43.5) (end 67.77 46.95) (width 0.6) (layer "B.Cu") (net 79))
-  (segment (start 87.77 43.5) (end 87.77 46.95) (width 0.6) (layer "B.Cu") (net 80))
-  (segment (start 107.77 43.5) (end 107.77 46.95) (width 0.6) (layer "B.Cu") (net 81))
-  (segment (start 127.77 43.5) (end 127.77 46.95) (width 0.6) (layer "B.Cu") (net 82))
-  (segment (start 147.77 43.5) (end 147.77 46.95) (width 0.6) (layer "B.Cu") (net 83))
-  (segment (start 167.77 43.5) (end 167.77 46.95) (width 0.6) (layer "B.Cu") (net 84))
-  (segment (start 187.77 43.5) (end 187.77 46.95) (width 0.6) (layer "B.Cu") (net 85))
-  (segment (start 207.77 43.5) (end 207.77 46.95) (width 0.6) (layer "B.Cu") (net 86))
-  (segment (start 227.77 43.5) (end 227.77 46.95) (width 0.6) (layer "B.Cu") (net 87))
-  (segment (start 247.77 43.5) (end 247.77 46.95) (width 0.6) (layer "B.Cu") (net 88))
   (zone (net 3) (net_name "GND") (layer "F.Cu") (hatch edge 0.508)
     (connect_pads (clearance 0.508))
