File: kicad/optocouplers-rewire/optocouplers.kicad_pcb (KiCad board)
At the start: 2 copper layers, 123 parts, among them Q1 PN2222A, Q2 PN2222A, Q3 PN2222A, Q4 PN2222A, Q5 PN2222A, Q6 PN2222A, Q7 PN2222A, Q8 PN2222A

Commit message: Place resistors R.R0 to R.R5
Parts:
- moved R.R5 133.1 mm to (116.5, 36.3), turned to 90 degrees
- moved R.R4 118.4 mm to (96.5, 36.3), turned to 90 degrees
- moved R.R3 97.4 mm to (76.5, 36.3), turned to 90 degrees
- moved R.R2 78.4 mm to (56.5, 36.3), turned to 90 degrees
- moved R.R1 59.3 mm to (36.5, 36.3), turned to 90 degrees
- moved R.R0 34.6 mm to (16.5, 36.3), turned to 90 degrees

Commit message: Simple connections between neighbours
Routing:
- net arduino_A1: track 0.00 -> 48.8 mm
- net arduino_A3: track 0.00 -> 48.7 mm
- net arduino_A5: track 0.00 -> 48.4 mm
- net arduino_A4: track 0.00 -> 48.2 mm
- net arduino_A0: track 0.00 -> 48.1 mm
- net arduino_A2: track 0.00 -> 48.1 mm
Changed lines of the file:
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@@
     )
   )
+  (segment (start 22.75 36.35) (end 21.23 37.87) (width 0.6) (layer "B.Cu") (net 5))
+  (segment (start 165.23 53.5) (end 163.08 51.35) (width 0.6) (layer "B.Cu") (net 5))
+  (segment (start 21.23 37.87) (end 21.23 38.5) (width 0.6) (layer "B.Cu") (net 5))
+  (segment (start 149.23 38.5) (end 147.08 36.35) (width 0.6) (layer "B.Cu") (net 5))
+  (segment (start 153.23 53.144416) (end 153.23 53.5) (width 0.6) (layer "B.Cu") (net 5))
+  (segment (start 155.024416 51.35) (end 153.23 53.144416) (width 0.6) (layer "B.Cu") (net 5))
+  (segment (start 33.23 53.144416) (end 33.23 53.5) (width 0.6) (layer "B.Cu") (net 5))
+  (segment (start 147.08 36.35) (end 143.024416 36.35) (width 0.6) (layer "B.Cu") (net 5))
+  (segment (start 143.024416 36.35) (end 141.23 38.144416) (width 0.6) (layer "B.Cu") (net 5))
+  (segment (start 29.23 38.5) (end 27.08 36.35) (width 0.6) (layer "B.Cu") (net 5))
+  (segment (start 27.08 36.35) (end 22.75 36.35) (width 0.6) (layer "B.Cu") (net 5))
+  (segment (start 43.08 51.35) (end 35.024416 51.35) (width 0.6) (layer "B.Cu") (net 5))
+  (segment (start 141.23 38.144416) (end 141.23 38.5) (width 0.6) (layer "B.Cu") (net 5))
+  (segment (start 163.08 51.35) (end 155.024416 51.35) (width 0.6) (layer "B.Cu") (net 5))
+  (segment (start 45.23 53.5) (end 43.08 51.35) (width 0.6) (layer "B.Cu") (net 5))
+  (segment (start 35.024416 51.35) (end 33.23 53.144416) (width 0.6) (layer "B.Cu") (net 5))
+  (segment (start 63.08 51.35) (end 54.35 51.35) (width 0.6) (layer "B.Cu") (net 6))
+  (segment (start 42.75 36.35) (end 41.23 37.87) (width 0.6) (layer "B.Cu") (net 6))
+  (segment (start 167.08 36.35) (end 162.45 36.35) (width 0.6) (layer "B.Cu") (net 6))
+  (segment (start 175.024416 51.35) (end 173.23 53.144416) (width 0.6) (layer "B.Cu") (net 6))
+  (segment (start 173.23 53.144416) (end 173.23 53.5) (width 0.6) (layer "B.Cu") (net 6))
+  (segment (start 161.23 37.57) (end 161.23 38.5) (width 0.6) (layer "B.Cu") (net 6))
+  (segment (start 41.23 37.87) (end 41.23 38.5) (width 0.6) (layer "B.Cu") (net 6))
+  (segment (start 169.23 38.5) (end 167.08 36.35) (width 0.6) (layer "B.Cu") (net 6))
+  (segment (start 49.23 38.5) (end 47.08 36.35) (width 0.6) (layer "B.Cu") (net 6))
+  (segment (start 162.45 36.35) (end 161.23 37.57) (width 0.6) (layer "B.Cu") (net 6))
+  (segment (start 53.23 52.47) (end 53.23 53.5) (width 0.6) (layer "B.Cu") (net 6))
+  (segment (start 65.23 53.5) (end 63.08 51.35) (width 0.6) (layer "B.Cu") (net 6))
+  (segment (start 185.23 53.5) (end 183.08 51.35) (width 0.6) (layer "B.Cu") (net 6))
+  (segment (start 54.35 51.35) (end 53.23 52.47) (width 0.6) (layer "B.Cu") (net 6))
+  (segment (start 47.08 36.35) (end 42.75 36.35) (width 0.6) (layer "B.Cu") (net 6))
+  (segment (start 183.08 51.35) (end 175.024416 51.35) (width 0.6) (layer "B.Cu") (net 6))
+  (segment (start 73.23 53.144416) (end 73.23 53.5) (width 0.6) (layer "B.Cu") (net 7))
+  (segment (start 61.23 37.97) (end 61.23 38.5) (width 0.6) (layer "B.Cu") (net 7))
+  (segment (start 69.23 38.5) (end 67.08 36.35) (width 0.6) (layer "B.Cu") (net 7))
+  (segment (start 83.08 51.35) (end 75.024416 51.35) (width 0.6) (layer "B.Cu") (net 7))
+  (segment (start 62.85 36.35) (end 61.23 37.97) (width 0.6) (layer "B.Cu") (net 7))
+  (segment (start 193.23 53.144416) (end 193.23 53.5) (width 0.6) (layer "B.Cu") (net 7))
+  (segment (start 189.23 38.5) (end 187.08 36.35) (width 0.6) (layer "B.Cu") (net 7))
+  (segment (start 183.024416 36.35) (end 181.23 38.144416) (width 0.6) (layer "B.Cu") (net 7))
+  (segment (start 181.23 38.144416) (end 181.23 38.5) (width 0.6) (layer "B.Cu") (net 7))
+  (segment (start 203.08 51.35) (end 195.024416 51.35) (width 0.6) (layer "B.Cu") (net 7))
+  (segment (start 195.024416 51.35) (end 193.23 53.144416) (width 0.6) (layer "B.Cu") (net 7))
+  (segment (start 75.024416 51.35) (end 73.23 53.144416) (width 0.6) (layer "B.Cu") (net 7))
+  (segment (start 205.23 53.5) (end 203.08 51.35) (width 0.6) (layer "B.Cu") (net 7))
+  (segment (start 85.23 53.5) (end 83.08 51.35) (width 0.6) (layer "B.Cu") (net 7))
+  (segment (start 187.08 36.35) (end 183.024416 36.35) (width 0.6) (layer "B.Cu") (net 7))
+  (segment (start 67.08 36.35) (end 62.85 36.35) (width 0.6) (layer "B.Cu") (net 7))
+  (segment (start 201.23 37.67) (end 201.23 38.5) (width 0.6) (layer "B.Cu") (net 8))
+  (segment (start 225.23 53.5) (end 223.08 51.35) (width 0.6) (layer "B.Cu") (net 8))
+  (segment (start 209.23 38.5) (end 207.08 36.35) (width 0.6) (layer "B.Cu") (net 8))
+  (segment (start 103.08 51.35) (end 95.024416 51.35) (width 0.6) (layer "B.Cu") (net 8))
+  (segment (start 213.23 53.144416) (end 213.23 53.5) (width 0.6) (layer "B.Cu") (net 8))
+  (segment (start 82.55 36.35) (end 81.23 37.67) (width 0.6) (layer "B.Cu") (net 8))
+  (segment (start 87.43 36.35) (end 82.55 36.35) (width 0.6) (layer "B.Cu") (net 8))
+  (segment (start 105.23 53.5) (end 103.08 51.35) (width 0.6) (layer "B.Cu") (net 8))
+  (segment (start 215.024416 51.35) (end 213.23 53.144416) (width 0.6) (layer "B.Cu") (net 8))
+  (segment (start 89.23 38.15) (end 87.43 36.35) (width 0.6) (layer "B.Cu") (net 8))
+  (segment (start 93.23 53.144416) (end 93.23 53.5) (width 0.6) (layer "B.Cu") (net 8))
+  (segment (start 202.55 36.35) (end 201.23 37.67) (width 0.6) (layer "B.Cu") (net 8))
+  (segment (start 223.08 51.35) (end 215.024416 51.35) (width 0.6) (layer "B.Cu") (net 8))
+  (segment (start 207.08 36.35) (end 202.55 36.35) (width 0.6) (layer "B.Cu") (net 8))
+  (segment (start 95.024416 51.35) (end 93.23 53.144416) (width 0.6) (layer "B.Cu") (net 8))
+  (segment (start 81.23 37.67) (end 81.23 38.5) (width 0.6) (layer "B.Cu") (net 8))
+  (segment (start 89.23 38.5) (end 89.23 38.15) (width 0.6) (layer "B.Cu") (net 8))
+  (segment (start 113.23 52.97) (end 113.23 53.5) (width 0.6) (layer "B.Cu") (net 9))
+  (segment (start 245.23 53.5) (end 243.08 51.35) (width 0.6) (layer "B.Cu") (net 9))
+  (segment (start 125.23 53.5) (end 123.08 51.35) (width 0.6) (layer "B.Cu") (net 9))
+  (segment (start 114.85 51.35) (end 113.23 52.97) (width 0.6) (layer "B.Cu") (net 9))
+  (segment (start 235.024416 51.35) (end 233.23 53.144416) (width 0.6) (layer "B.Cu") (net 9))
+  (segment (start 227.08 36.35) (end 222.85 36.35) (width 0.6) (layer "B.Cu") (net 9))
+  (segment (start 243.08 51.35) (end 235.024416 51.35) (width 0.6) (layer "B.Cu") (net 9))
+  (segment (start 103.024416 36.35) (end 101.23 38.144416) (width 0.6) (layer "B.Cu") (net 9))
+  (segment (start 109.23 38.5) (end 107.08 36.35) (width 0.6) (layer "B.Cu") (net 9))
+  (segment (start 233.23 53.144416) (end 233.23 53.5) (width 0.6) (layer "B.Cu") (net 9))
+  (segment (start 222.85 36.35) (end 221.23 37.97) (width 0.6) (layer "B.Cu") (net 9))
+  (segment (start 107.08 36.35) (end 103.024416 36.35) (width 0.6) (layer "B.Cu") (net 9))
+  (segment (start 123.08 51.35) (end 114.85 51.35) (width 0.6) (layer "B.Cu") (net 9))
+  (segment (start 101.23 38.144416) (end 101.23 38.5) (width 0.6) (layer "B.Cu") (net 9))
+  (segment (start 221.23 37.97) (end 221.23 38.5) (width 0.6) (layer "B.Cu") (net 9))
+  (segment (start 229.23 38.5) (end 227.08 36.35) (width 0.6) (layer "B.Cu") (net 9))
+  (segment (start 145.23 53.5) (end 143.08 51.35) (width 0.6) (layer "B.Cu") (net 10))
+  (segment (start 242.25 36.35) (end 241.23 37.37) (width 0.6) (layer "B.Cu") (net 10))
+  (segment (start 123.024416 36.35) (end 121.23 38.144416) (width 0.6) (layer "B.Cu") (net 10))
+  (segment (start 261.23 38.5) (end 259.08 36.35) (width 0.6) (layer "B.Cu") (net 10))
+  (segment (start 133.23 53.144416) (end 133.23 53.5) (width 0.6) (layer "B.Cu") (net 10))
+  (segment (start 143.08 51.35) (end 135.024416 51.35) (width 0.6) (layer "B.Cu") (net 10))
+  (segment (start 249.23 38.5) (end 247.08 36.35) (width 0.6) (layer "B.Cu") (net 10))
+  (segment (start 259.08 36.35) (end 251.024416 36.35) (width 0.6) (layer "B.Cu") (net 10))
+  (segment (start 249.23 38.144416) (end 249.23 38.5) (width 0.6) (layer "B.Cu") (net 10))
+  (segment (start 241.23 37.37) (end 241.23 38.5) (width 0.6) (layer "B.Cu") (net 10))
+  (segment (start 251.024416 36.35) (end 249.23 38.144416) (width 0.6) (layer "B.Cu") (net 10))
+  (segment (start 129.23 38.5) (end 127.08 36.35) (width 0.6) (layer "B.Cu") (net 10))
+  (segment (start 247.08 36.35) (end 242.25 36.35) (width 0.6) (layer "B.Cu") (net 10))
+  (segment (start 121.23 38.144416) (end 121.23 38.5) (width 0.6) (layer "B.Cu") (net 10))
+  (segment (start 127.08 36.35) (end 123.024416 36.35) (width 0.6) (layer "B.Cu") (net 10))
+  (segment (start 135.024416 51.35) (end 133.23 53.144416) (width 0.6) (layer "B.Cu") (net 10))
   (zone (net 3) (net_name "GND") (layer "F.Cu") (hatch edge 0.508)
     (connect_pads (clearance 0.508))

Commit message: 5V line
Routing:
- net +5V: track 0.00 -> 467.3 mm
Changed lines of the file:
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@@
     )
   )
+  (segment (start 35.77 49.75) (end 255.77 49.75) (width 0.6) (layer "B.Cu") (net 4))
+  (segment (start 16.5 34.75) (end 263.77 34.75) (width 0.6) (layer "B.Cu") (net 4))
   (segment (start 22.75 36.35) (end 21.23 37.87) (width 0.6) (layer "B.Cu") (net 5))
   (segment (start 165.23 53.5) (end 163.08 51.35) (width 0.6) (layer "B.Cu") (net 5))

Commit message: Add some lines
Routing:
- net Net-(Q8-Pad3): track 0.00 -> 114.3 mm
- net Net-(Q6-Pad3): track 0.00 -> 103.1 mm
- net Net-(Q4-Pad3): track 0.00 -> 103.1 mm
- net Net-(Q7-Pad3): track 0.00 -> 103.1 mm
- net Net-(Q3-Pad3): track 0.00 -> 103.1 mm
- net Net-(Q5-Pad3): track 0.00 -> 102.9 mm
- net arduino_A5: track 48.4 -> 73.7 mm
- net arduino_A3: track 48.7 -> 53.7 mm
- net arduino_A0: track 48.1 -> 53.1 mm
- net arduino_A4: track 48.2 -> 53.2 mm
- net arduino_A2: track 48.1 -> 53.1 mm
- net arduino_A1: track 48.8 -> 53.8 mm
Changed lines of the file:
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@@
   (segment (start 43.08 51.35) (end 35.024416 51.35) (width 0.6) (layer "B.Cu") (net 5))
   (segment (start 141.23 38.144416) (end 141.23 38.5) (width 0.6) (layer "B.Cu") (net 5))
+  (segment (start 16.5 37.85) (end 20.58 37.85) (width 0.6) (layer "B.Cu") (net 5))
   (segment (start 163.08 51.35) (end 155.024416 51.35) (width 0.6) (layer "B.Cu") (net 5))
   (segment (start 45.23 53.5) (end 43.08 51.35) (width 0.6) (layer "B.Cu") (net 5))
+  (segment (start 20.58 37.85) (end 21.23 38.5) (width 0.6) (layer "B.Cu") (net 5))
   (segment (start 35.024416 51.35) (end 33.23 53.144416) (width 0.6) (layer "B.Cu") (net 5))
   (segment (start 63.08 51.35) (end 54.35 51.35) (width 0.6) (layer "B.Cu") (net 6))
@@
   (segment (start 53.23 52.47) (end 53.23 53.5) (width 0.6) (layer "B.Cu") (net 6))
   (segment (start 65.23 53.5) (end 63.08 51.35) (width 0.6) (layer "B.Cu") (net 6))
+  (segment (start 36.5 37.85) (end 40.58 37.85) (width 0.6) (layer "B.Cu") (net 6))
+  (segment (start 40.58 37.85) (end 41.23 38.5) (width 0.6) (layer "B.Cu") (net 6))
   (segment (start 185.23 53.5) (end 183.08 51.35) (width 0.6) (layer "B.Cu") (net 6))
   (segment (start 54.35 51.35) (end 53.23 52.47) (width 0.6) (layer "B.Cu") (net 6))
@@
   (segment (start 62.85 36.35) (end 61.23 37.97) (width 0.6) (layer "B.Cu") (net 7))
   (segment (start 193.23 53.144416) (end 193.23 53.5) (width 0.6) (layer "B.Cu") (net 7))
+  (segment (start 56.5 37.85) (end 60.58 37.85) (width 0.6) (layer "B.Cu") (net 7))
   (segment (start 189.23 38.5) (end 187.08 36.35) (width 0.6) (layer "B.Cu") (net 7))
   (segment (start 183.024416 36.35) (end 181.23 38.144416) (width 0.6) (layer "B.Cu") (net 7))
@@
   (segment (start 195.024416 51.35) (end 193.23 53.144416) (width 0.6) (layer "B.Cu") (net 7))
   (segment (start 75.024416 51.35) (end 73.23 53.144416) (width 0.6) (layer "B.Cu") (net 7))
+  (segment (start 60.58 37.85) (end 61.23 38.5) (width 0.6) (layer "B.Cu") (net 7))
   (segment (start 205.23 53.5) (end 203.08 51.35) (width 0.6) (layer "B.Cu") (net 7))
   (segment (start 85.23 53.5) (end 83.08 51.35) (width 0.6) (layer "B.Cu") (net 7))
@@
   (segment (start 93.23 53.144416) (end 93.23 53.5) (width 0.6) (layer "B.Cu") (net 8))
   (segment (start 202.55 36.35) (end 201.23 37.67) (width 0.6) (layer "B.Cu") (net 8))
+  (segment (start 80.58 37.85) (end 81.23 38.5) (width 0.6) (layer "B.Cu") (net 8))
+  (segment (start 76.5 37.85) (end 80.58 37.85) (width 0.6) (layer "B.Cu") (net 8))
   (segment (start 223.08 51.35) (end 215.024416 51.35) (width 0.6) (layer "B.Cu") (net 8))
   (segment (start 207.08 36.35) (end 202.55 36.35) (width 0.6) (layer "B.Cu") (net 8))
@@
   (segment (start 113.23 52.97) (end 113.23 53.5) (width 0.6) (layer "B.Cu") (net 9))
   (segment (start 245.23 53.5) (end 243.08 51.35) (width 0.6) (layer "B.Cu") (net 9))
+  (segment (start 100.58 37.85) (end 101.23 38.5) (width 0.6) (layer "B.Cu") (net 9))
   (segment (start 125.23 53.5) (end 123.08 51.35) (width 0.6) (layer "B.Cu") (net 9))
+  (segment (start 96.5 37.85) (end 100.58 37.85) (width 0.6) (layer "B.Cu") (net 9))
   (segment (start 114.85 51.35) (end 113.23 52.97) (width 0.6) (layer "B.Cu") (net 9))
   (segment (start 235.024416 51.35) (end 233.23 53.144416) (width 0.6) (layer "B.Cu") (net 9))
@@
   (segment (start 242.25 36.35) (end 241.23 37.37) (width 0.6) (layer "B.Cu") (net 10))
   (segment (start 123.024416 36.35) (end 121.23 38.144416) (width 0.6) (layer "B.Cu") (net 10))
+  (segment (start 253.23 51.65) (end 253.58 51.3) (width 0.6) (layer "B.Cu") (net 10))
   (segment (start 261.23 38.5) (end 259.08 36.35) (width 0.6) (layer "B.Cu") (net 10))
+  (segment (start 116.5 37.85) (end 120.58 37.85) (width 0.6) (layer "B.Cu") (net 10))
   (segment (start 133.23 53.144416) (end 133.23 53.5) (width 0.6) (layer "B.Cu") (net 10))
   (segment (start 143.08 51.35) (end 135.024416 51.35) (width 0.6) (layer "B.Cu") (net 10))
+  (segment (start 253.23 53.5) (end 253.23 51.65) (width 0.6) (layer "B.Cu") (net 10))
   (segment (start 249.23 38.5) (end 247.08 36.35) (width 0.6) (layer "B.Cu") (net 10))
   (segment (start 259.08 36.35) (end 251.024416 36.35) (width 0.6) (layer "B.Cu") (net 10))
+  (segment (start 120.58 37.85) (end 121.23 38.5) (width 0.6) (layer "B.Cu") (net 10))
   (segment (start 249.23 38.144416) (end 249.23 38.5) (width 0.6) (layer "B.Cu") (net 10))
   (segment (start 241.23 37.37) (end 241.23 38.5) (width 0.6) (layer "B.Cu") (net 10))
   (segment (start 251.024416 36.35) (end 249.23 38.144416) (width 0.6) (layer "B.Cu") (net 10))
+  (segment (start 256.871346 51.3) (end 261.23 46.941346) (width 0.6) (layer "B.Cu") (net 10))
+  (segment (start 261.23 46.941346) (end 261.23 38.5) (width 0.6) (layer "B.Cu") (net 10))
   (segment (start 129.23 38.5) (end 127.08 36.35) (width 0.6) (layer "B.Cu") (net 10))
   (segment (start 247.08 36.35) (end 242.25 36.35) (width 0.6) (layer "B.Cu") (net 10))
+  (segment (start 253.58 51.3) (end 256.871346 51.3) (width 0.6) (layer "B.Cu") (net 10))
   (segment (start 121.23 38.144416) (end 121.23 38.5) (width 0.6) (layer "B.Cu") (net 10))
   (segment (start 127.08 36.35) (end 123.024416 36.35) (width 0.6) (layer "B.Cu") (net 10))
   (segment (start 135.024416 51.35) (end 133.23 53.144416) (width 0.6) (layer "B.Cu") (net 10))
+  (segment (start 21.23 28.5) (end 21.23 26.65) (width 0.6) (layer "B.Cu") (net 22))
+  (segment (start 21.23 26.65) (end 21.793525 26.086475) (width 0.6) (layer "B.Cu") (net 22))
+  (segment (start 118.816475 26.086475) (end 121.23 28.5) (width 0.6) (layer "B.Cu") (net 22))
+  (segment (start 21.793525 26.086475) (end 118.816475 26.086475) (width 0.6) (layer "B.Cu") (net 22))
+  (segment (start 238.816475 26.086475) (end 241.23 28.5) (width 0.6) (layer "B.Cu") (net 23))
+  (segment (start 141.23 26.65) (end 141.793525 26.086475) (width 0.6) (layer "B.Cu") (net 23))
+  (segment (start 141.23 28.5) (end 141.23 26.65) (width 0.6) (layer "B.Cu") (net 23))
+  (segment (start 141.793525 26.086475) (end 238.816475 26.086475) (width 0.6) (layer "B.Cu") (net 23))
+  (segment (start 33.23 43.5) (end 33.23 41.65) (width 0.6) (layer "B.Cu") (net 26))
+  (segment (start 33.53 41.35) (end 131.08 41.35) (width 0.6) (layer "B.Cu") (net 26))
+  (segment (start 131.08 41.35) (end 133.23 43.5) (width 0.6) (layer "B.Cu") (net 26))
+  (segment (start 33.23 41.65) (end 33.53 41.35) (width 0.6) (layer "B.Cu") (net 26))
+  (segment (start 250.816475 41.086475) (end 253.23 43.5) (width 0.6) (layer "B.Cu") (net 27))
+  (segment (start 153.23 41.65) (end 153.793525 41.086475) (width 0.6) (layer "B.Cu") (net 27))
+  (segment (start 153.23 43.5) (end 153.23 41.65) (width 0.6) (layer "B.Cu") (net 27))
+  (segment (start 153.793525 41.086475) (end 250.816475 41.086475) (width 0.6) (layer "B.Cu") (net 27))
+  (segment (start 45.23 45.35) (end 45.793525 45.913525) (width 0.6) (layer "F.Cu") (net 30))
+  (segment (start 45.793525 45.913525) (end 142.816475 45.913525) (width 0.6) (layer "F.Cu") (net 30))
+  (segment (start 142.816475 45.913525) (end 145.23 43.5) (width 0.6) (layer "F.Cu") (net 30))
+  (segment (start 45.23 43.5) (end 45.23 45.35) (width 0.6) (layer "F.Cu") (net 30))
+  (segment (start 249.4 45.7) (end 251.43 43.67) (width 0.6) (layer "F.Cu") (net 31))
+  (segment (start 258.3 40.5) (end 258.3 31.43) (width 0.6) (layer "F.Cu") (net 31))
+  (segment (start 258.3 31.43) (end 261.23 28.5) (width 0.6) (layer "F.Cu") (net 31))
+  (segment (start 253.334416 40.5) (end 258.3 40.5) (width 0.6) (layer "F.Cu") (net 31))
+  (segment (start 165.23 45.35) (end 165.793525 45.913525) (width 0.6) (layer "F.Cu") (net 31))
+  (segment (start 251.43 42.404416) (end 253.334416 40.5) (width 0.6) (layer "F.Cu") (net 31))
+  (segment (start 242.816475 45.913525) (end 245.23 43.5) (width 0.6) (layer "F.Cu") (net 31))
+  (segment (start 165.793525 45.913525) (end 242.816475 45.913525) (width 0.6) (layer "F.Cu") (net 31))
+  (segment (start 245.23 43.5) (end 245.23 45.35) (width 0.6) (layer "F.Cu") (net 31))
+  (segment (start 165.23 43.5) (end 165.23 45.35) (width 0.6) (layer "F.Cu") (net 31))
+  (segment (start 245.23 45.35) (end 245.58 45.7) (width 0.6) (layer "F.Cu") (net 31))
+  (segment (start 251.43 43.67) (end 251.43 42.404416) (width 0.6) (layer "F.Cu") (net 31))
+  (segment (start 245.58 45.7) (end 249.4 45.7) (width 0.6) (layer "F.Cu") (net 31))
   (zone (net 3) (net_name "GND") (layer "F.Cu") (hatch edge 0.508)
     (connect_pads (clearance 0.508))

Commit message: More lines
Routing:
- net Net-(Q1-Pad3): track 0.00 -> 103.1 mm
- net Net-(Q2-Pad3): track 0.00 -> 102.2 mm
- net arduino_A0: track 53.1 -> 69.8 mm
Changed lines of the file:
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@@
     )
   )
+  (segment (start 126.816475 26.086475) (end 129.23 28.5) (width 0.6) (layer "F.Cu") (net 2))
+  (segment (start 29.793525 26.086475) (end 126.816475 26.086475) (width 0.6) (layer "F.Cu") (net 2))
+  (segment (start 29.23 26.65) (end 29.793525 26.086475) (width 0.6) (layer "F.Cu") (net 2))
+  (segment (start 29.23 28.5) (end 29.23 26.65) (width 0.6) (layer "F.Cu") (net 2))
   (segment (start 35.77 49.75) (end 255.77 49.75) (width 0.6) (layer "B.Cu") (net 4))
   (segment (start 16.5 34.75) (end 263.77 34.75) (width 0.6) (layer "B.Cu") (net 4))
@@
   (segment (start 21.23 37.87) (end 21.23 38.5) (width 0.6) (layer "B.Cu") (net 5))
   (segment (start 149.23 38.5) (end 147.08 36.35) (width 0.6) (layer "B.Cu") (net 5))
+  (segment (start 33.23 53.5) (end 29.23 49.5) (width 0.6) (layer "B.Cu") (net 5))
+  (segment (start 29.23 49.5) (end 29.23 38.5) (width 0.6) (layer "B.Cu") (net 5))
   (segment (start 153.23 53.144416) (end 153.23 53.5) (width 0.6) (layer "B.Cu") (net 5))
   (segment (start 155.024416 51.35) (end 153.23 53.144416) (width 0.6) (layer "B.Cu") (net 5))
@@
   (segment (start 127.08 36.35) (end 123.024416 36.35) (width 0.6) (layer "B.Cu") (net 10))
   (segment (start 135.024416 51.35) (end 133.23 53.144416) (width 0.6) (layer "B.Cu") (net 10))
+  (segment (start 246.816475 26.086475) (end 249.23 28.5) (width 0.6) (layer "F.Cu") (net 19))
+  (segment (start 151.287941 26.086475) (end 246.816475 26.086475) (width 0.6) (layer "F.Cu") (net 19))
+  (segment (start 149.23 28.144416) (end 151.287941 26.086475) (width 0.6) (layer "F.Cu") (net 19))
+  (segment (start 149.23 28.5) (end 149.23 28.144416) (width 0.6) (layer "F.Cu") (net 19))
   (segment (start 21.23 28.5) (end 21.23 26.65) (width 0.6) (layer "B.Cu") (net 22))
   (segment (start 21.23 26.65) (end 21.793525 26.086475) (width 0.6) (layer "B.Cu") (net 22))

Commit message: Move optocouplers to the correct place, shrink the board
Parts:
- moved R.B5 21.0 mm to (128.3, 12.7)
- moved R.D4 21.0 mm to (132.3, 27.7)
- moved R.A0 21.0 mm to (36.3, 12.7)
- moved R.A1 21.0 mm to (56.3, 12.7)
- moved R.A10 21.0 mm to (236.3, 12.7)
- moved R.A2 21.0 mm to (76.3, 12.7)
- moved R.A3 21.0 mm to (96.3, 12.7)
- moved R.A4 21.0 mm to (116.3, 12.7)
- moved R.A5 21.0 mm to (136.3, 12.7)
- moved R.A6 21.0 mm to (156.3, 12.7)
- moved R.A7 21.0 mm to (176.3, 12.7)
- moved R.A8 21.0 mm to (196.3, 12.7)
- moved R.A9 21.0 mm to (216.3, 12.7)
- moved R.B0 21.0 mm to (28.3, 12.7)
- moved R.B1 21.0 mm to (48.3, 12.7)
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Routing:
- net Net-(Q1-Pad3): track 103.1 -> 111.4 mm
- net Net-(Q2-Pad3): track 102.2 -> 110.5 mm
- net Net-(Q3-Pad3): track 103.1 -> 111.2 mm
- net Net-(Q4-Pad3): track 103.1 -> 111.2 mm
- net Net-(Q5-Pad3): track 102.9 -> 110.5 mm
- net Net-(Q8-Pad3): track 114.3 -> 120.5 mm
- net Net-(U.A6-Pad1): track 0.00 -> 3.15 mm
- net Net-(R.B9-Pad1): track 0.00 -> 3.15 mm
- net Net-(R.B8-Pad1): track 0.00 -> 3.15 mm
- net Net-(R.B7-Pad1): track 0.00 -> 3.15 mm
- net Net-(R.B6-Pad1): track 0.00 -> 3.15 mm
- net Net-(R.B5-Pad1): track 0.00 -> 3.15 mm
- net Net-(R.B4-Pad1): track 0.00 -> 3.15 mm
- net Net-(R.B3-Pad1): track 0.00 -> 3.15 mm
- net Net-(R.B2-Pad1): track 0.00 -> 3.15 mm
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Other:
- board outline added: 294 x 50 mm
- rule pad_to_mask_clearance: 0.2 -> 0
