File: kicad/optocouplers-rewire/optocouplers.kicad_pcb (KiCad board)
At the start: 2 copper layers, 294 x 50 mm, 123 parts, among them Q1 PN2222A, Q2 PN2222A, Q3 PN2222A, Q4 PN2222A, Q5 PN2222A, Q6 PN2222A, Q7 PN2222A, Q8 PN2222A

Commit message: optocouplers, continue wiring
Parts:
- Q1, Q2, Q3, Q4, Q5, Q6, Q7, Q8: footprint Package_TO_SOT_THT:TO-92L_HandSolder -> Package_TO_SOT_THT:TO-92_Inline_Wide
- moved Q2 236.6 mm to (265.0, 45.0), turned to 90 degrees
- moved R2 232.2 mm to (260.9, 40.9), turned to -90 degrees
- moved Q4 212.6 mm to (255.0, 45.0), turned to 90 degrees
- moved R4 208.2 mm to (250.9, 40.9), turned to -90 degrees
- moved Q6 188.6 mm to (245.0, 45.0), turned to 90 degrees
- moved R6 184.2 mm to (240.9, 40.9), turned to -90 degrees
- moved Q8 164.6 mm to (235.0, 45.0), turned to 90 degrees
- moved R8 160.2 mm to (230.9, 40.9), turned to -90 degrees
- moved Conn1 18.1 mm to (70.0, 41.0)
- moved R7 13.0 mm to (50.9, 41.0), turned to 90 degrees
- moved Q7 9.19 mm to (55.0, 42.0), turned to 90 degrees
- moved R5 9.04 mm to (40.9, 41.0), turned to 90 degrees
- moved Q5 5.70 mm to (45.0, 42.0), turned to 90 degrees
- moved R3 5.22 mm to (30.9, 41.0), turned to 90 degrees
- moved Q1 4.95 mm to (25.0, 42.0), turned to 90 degrees
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Routing:
- net arduino_D6: track 0.00 -> 182.2 mm
- net arduino_D8: track 0.00 -> 166.1 mm
- net arduino_D10: track 0.00 -> 150.0 mm
- net arduino_D12: track 0.00 -> 133.9 mm
- net Net-(Q4-Pad3): track 111.2 -> 179.3 mm, vias 0 -> 1
- net arduino_D5: track 0.00 -> 65.3 mm
- net arduino_D7: track 0.00 -> 60.4 mm, vias 0 -> 1
- net arduino_D9: track 0.00 -> 55.4 mm, vias 0 -> 1
- net Net-(Q2-Pad3): track 110.5 -> 165.7 mm
- net arduino_D11: track 0.00 -> 50.5 mm, vias 0 -> 1
- net Net-(Q1-Pad3): track 111.4 -> 153.7 mm
- net arduino_A3: track 53.7 -> 87.0 mm
- net arduino_A4: track 53.2 -> 86.5 mm
- net arduino_A1: track 53.8 -> 87.2 mm
- net arduino_A2: track 53.1 -> 86.4 mm
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
Commit message: Move the whole optocouplers board a bit up, finish tracing
Parts:
- moved Conn1 2.00 mm to (70.0, 39.0)
- moved Q1 2.00 mm to (25.0, 40.0)
- moved Q2 2.00 mm to (265.0, 43.0)
- moved Q3 2.00 mm to (35.0, 40.0)
- moved Q4 2.00 mm to (255.0, 43.0)
- moved Q5 2.00 mm to (45.0, 40.0)
- moved Q6 2.00 mm to (245.0, 43.0)
- moved Q7 2.00 mm to (55.0, 40.0)
- moved Q8 2.00 mm to (235.0, 43.0)
- moved R.A0 2.00 mm to (36.3, 10.7)
- moved R.A1 2.00 mm to (56.3, 10.7)
- moved R.A10 2.00 mm to (236.3, 10.7)
- moved R.A11 2.00 mm to (256.3, 10.7)
- moved R.A2 2.00 mm to (76.3, 10.7)
- moved R.A3 2.00 mm to (96.3, 10.7)
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Routing:
- net arduino_A5: track 90.3 -> 322.2 mm, vias 0 -> 1
- net arduino_A4: track 86.5 -> 272.9 mm, vias 0 -> 2
- net arduino_A1: track 87.2 -> 253.6 mm, vias 0 -> 1
- net arduino_A3: track 87.0 -> 247.6 mm, vias 0 -> 2
- net arduino_A2: track 86.4 -> 239.2 mm, vias 0 -> 3
- net arduino_A0: track 86.4 -> 218.7 mm, vias 0 -> 2
- net +5V: track 467.3 -> 503.3 mm, vias 0 -> 2
- net Net-(Q4-Pad3): track 179.3 -> 153.8 mm
- net Net-(Q6-Pad3): track 122.5 -> 132.3 mm
- net Net-(Q1-Pad3): track 153.7 -> 162.9 mm, vias 0 -> 1
- net Net-(Q2-Pad3): track 165.7 -> 174.0 mm, vias 0 -> 1
- net GND: vias 0 -> 65
