File: kicad/optocouplers-rewire/optocouplers.kicad_sch (KiCad schematic)
At the start: 119 parts

Commit message: Update components
Parts:
- Conn1: value (none) -> Conn_02x13_Odd_Even; footprint (none) -> Connector_IDC:IDC-Header_2x13_P2.54mm_Vertical
- Q1, Q2, Q3, Q4, Q5, Q6, Q7, Q8: value (none) -> PN2222A; footprint (none) -> Package_TO_SOT_THT:TO-92L_HandSolder
- R.A0, R.A1, R.A10, R.A11, R.A2, R.A3, R.A4, R.A5, R.A6, R.A7, R.A8, R.A9, R.B0, R.B1, R.B10, R.B11, R.B12, R.B2, R.B3, R.B4, R.B5, R.B6, R.B7, R.B8, R.B9, R.C0, R.C1, R.C10, R.C11, R.C2, R.C3, R.C4, R.C5, R.C6, R.C7, R.C8, R.C9, R.D0, R.D1, R.D10, R.D2, R.D3, R.D4, R.D5, R.D6, R.D7, R.D8, R.D9: value (none) -> 270R; footprint (none) -> Resistor_SMD:R_1206_3216Metric_Pad1.30x1.75mm_HandSolder
- R1, R2, R3, R4, R5, R6, R7, R8: value (none) -> 1k; footprint (none) -> Resistor_SMD:R_1206_3216Metric_Pad1.30x1.75mm_HandSolder
- R_R0, R_R1, R_R2, R_R3, R_R4, R_R5: value (none) -> 2k; footprint (none) -> Resistor_SMD:R_1206_3216Metric_Pad1.30x1.75mm_HandSolder
- U.A0, U.A1, U.A10, U.A11, U.A2, U.A3, U.A4, U.A5, U.A6, U.A7, U.A8, U.A9, U.B0, U.B1, U.B10, U.B11, U.B12, U.B2, U.B3, U.B4, U.B5, U.B6, U.B7, U.B8, U.B9, U.C0, U.C1, U.C10, U.C11, U.C2, U.C3, U.C4, U.C5, U.C6, U.C7, U.C8, U.C9, U.D0, U.D1, U.D10, U.D2, U.D3, U.D4, U.D5, U.D6, U.D7, U.D8, U.D9: value (none) -> ITR9608; footprint (none) -> ITR9608:ITR9608

Commit message: rename some components in schematic
Parts:
- renumbered R_R0 to R.R0, R_R1 to R.R1, R_R2 to R.R2, R_R3 to R.R3, R_R4 to R.R4, R_R5 to R.R5
Changed lines of the file:
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@@
   (symbol (lib_id "Device:R") (at 392.43 30.48 270) (unit 1)
     (in_bom yes) (on_board yes)
-    (property "Reference" "R_R0" (id 0) (at 392.43 33.02 90))
+    (property "Reference" "R.R0" (id 0) (at 392.43 33.02 90))
     (property "Value" "2k" (id 1) (at 392.43 30.48 90))
     (property "Footprint" "Resistor_SMD:R_1206_3216Metric_Pad1.30x1.75mm_HandSolder" (id 2) (at 392.43 28.702 90)
@@
   (symbol (lib_id "Device:R") (at 392.43 43.18 270) (unit 1)
     (in_bom yes) (on_board yes)
-    (property "Reference" "R_R1" (id 0) (at 392.43 45.72 90))
+    (property "Reference" "R.R1" (id 0) (at 392.43 45.72 90))
     (property "Value" "2k" (id 1) (at 392.43 43.18 90))
     (property "Footprint" "Resistor_SMD:R_1206_3216Metric_Pad1.30x1.75mm_HandSolder" (id 2) (at 392.43 41.402 90)
@@
   (symbol (lib_id "Device:R") (at 392.43 55.88 270) (unit 1)
     (in_bom yes) (on_board yes)
-    (property "Reference" "R_R2" (id 0) (at 392.43 58.42 90))
+    (property "Reference" "R.R2" (id 0) (at 392.43 58.42 90))
     (property "Value" "2k" (id 1) (at 392.43 55.88 90))
     (property "Footprint" "Resistor_SMD:R_1206_3216Metric_Pad1.30x1.75mm_HandSolder" (id 2) (at 392.43 54.102 90)
@@
   (symbol (lib_id "Device:R") (at 392.43 68.58 270) (unit 1)
     (in_bom yes) (on_board yes)
-    (property "Reference" "R_R3" (id 0) (at 392.43 71.12 90))
+    (property "Reference" "R.R3" (id 0) (at 392.43 71.12 90))
     (property "Value" "2k" (id 1) (at 392.43 68.58 90))
     (property "Footprint" "Resistor_SMD:R_1206_3216Metric_Pad1.30x1.75mm_HandSolder" (id 2) (at 392.43 66.802 90)
@@
   (symbol (lib_id "Device:R") (at 392.43 81.28 270) (unit 1)
     (in_bom yes) (on_board yes)
-    (property "Reference" "R_R4" (id 0) (at 392.43 83.82 90))
+    (property "Reference" "R.R4" (id 0) (at 392.43 83.82 90))
     (property "Value" "2k" (id 1) (at 392.43 81.28 90))
     (property "Footprint" "Resistor_SMD:R_1206_3216Metric_Pad1.30x1.75mm_HandSolder" (id 2) (at 392.43 79.502 90)
@@
   (symbol (lib_id "Device:R") (at 392.43 93.98 270) (unit 1)
     (in_bom yes) (on_board yes)
-    (property "Reference" "R_R5" (id 0) (at 392.43 96.52 90))
+    (property "Reference" "R.R5" (id 0) (at 392.43 96.52 90))
     (property "Value" "2k" (id 1) (at 392.43 93.98 90))
     (property "Footprint" "Resistor_SMD:R_1206_3216Metric_Pad1.30x1.75mm_HandSolder" (id 2) (at 392.43 92.202 90)
@@
     )
     (path "/00000000-0000-0000-0000-00005db27a45"
-      (reference "R_R0") (unit 1) (value "2k") (footprint "Resistor_SMD:R_1206_3216Metric_Pad1.30x1.75mm_HandSolder")
+      (reference "R.R0") (unit 1) (value "2k") (footprint "Resistor_SMD:R_1206_3216Metric_Pad1.30x1.75mm_HandSolder")
     )
     (path "/00000000-0000-0000-0000-00005db2c8a5"
-      (reference "R_R1") (unit 1) (value "2k") (footprint "Resistor_SMD:R_1206_3216Metric_Pad1.30x1.75mm_HandSolder")
+      (reference "R.R1") (unit 1) (value "2k") (footprint "Resistor_SMD:R_1206_3216Metric_Pad1.30x1.75mm_HandSolder")
     )
     (path "/00000000-0000-0000-0000-00005db2ed55"
-      (reference "R_R2") (unit 1) (value "2k") (footprint "Resistor_SMD:R_1206_3216Metric_Pad1.30x1.75mm_HandSolder")
+      (reference "R.R2") (unit 1) (value "2k") (footprint "Resistor_SMD:R_1206_3216Metric_Pad1.30x1.75mm_HandSolder")
     )
     (path "/00000000-0000-0000-0000-00005db31435"
-      (reference "R_R3") (unit 1) (value "2k") (footprint "Resistor_SMD:R_1206_3216Metric_Pad1.30x1.75mm_HandSolder")
+      (reference "R.R3") (unit 1) (value "2k") (footprint "Resistor_SMD:R_1206_3216Metric_Pad1.30x1.75mm_HandSolder")
     )
     (path "/00000000-0000-0000-0000-00005db3377d"
-      (reference "R_R4") (unit 1) (value "2k") (footprint "Resistor_SMD:R_1206_3216Metric_Pad1.30x1.75mm_HandSolder")
+      (reference "R.R4") (unit 1) (value "2k") (footprint "Resistor_SMD:R_1206_3216Metric_Pad1.30x1.75mm_HandSolder")
     )
     (path "/00000000-0000-0000-0000-00005db35c7d"
-      (reference "R_R5") (unit 1) (value "2k") (footprint "Resistor_SMD:R_1206_3216Metric_Pad1.30x1.75mm_HandSolder")
+      (reference "R.R5") (unit 1) (value "2k") (footprint "Resistor_SMD:R_1206_3216Metric_Pad1.30x1.75mm_HandSolder")
     )
     (path "/00000000-0000-0000-0000-0000598263bf"

Commit message: optocouplers: change footprints
Parts:
- Q1, Q2, Q3, Q4, Q5, Q6, Q7, Q8: footprint Package_TO_SOT_THT:TO-92L_HandSolder -> Package_TO_SOT_THT:TO-92_Inline_Wide
Changed lines of the file:
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@@
       (effects (font (size 1.27 1.27)) (justify left))
     )
-    (property "Footprint" "Package_TO_SOT_THT:TO-92L_HandSolder" (id 2) (at 29.845 101.6 0)
+    (property "Footprint" "Package_TO_SOT_THT:TO-92_Inline_Wide" (id 2) (at 29.845 101.6 0)
       (effects (font (size 1.27 1.27) italic) (justify left) hide)
     )
@@
       (effects (font (size 1.27 1.27)) (justify left))
     )
-    (property "Footprint" "Package_TO_SOT_THT:TO-92L_HandSolder" (id 2) (at 75.565 101.6 0)
+    (property "Footprint" "Package_TO_SOT_THT:TO-92_Inline_Wide" (id 2) (at 75.565 101.6 0)
       (effects (font (size 1.27 1.27) italic) (justify left) hide)
     )
@@
       (effects (font (size 1.27 1.27)) (justify left))
     )
-    (property "Footprint" "Package_TO_SOT_THT:TO-92L_HandSolder" (id 2) (at 121.285 101.6 0)
+    (property "Footprint" "Package_TO_SOT_THT:TO-92_Inline_Wide" (id 2) (at 121.285 101.6 0)
       (effects (font (size 1.27 1.27) italic) (justify left) hide)
     )
@@
       (effects (font (size 1.27 1.27)) (justify left))
     )
-    (property "Footprint" "Package_TO_SOT_THT:TO-92L_HandSolder" (id 2) (at 167.005 101.6 0)
+    (property "Footprint" "Package_TO_SOT_THT:TO-92_Inline_Wide" (id 2) (at 167.005 101.6 0)
       (effects (font (size 1.27 1.27) italic) (justify left) hide)
     )
@@
       (effects (font (size 1.27 1.27)) (justify left))
     )
-    (property "Footprint" "Package_TO_SOT_THT:TO-92L_HandSolder" (id 2) (at 212.725 101.6 0)
+    (property "Footprint" "Package_TO_SOT_THT:TO-92_Inline_Wide" (id 2) (at 212.725 101.6 0)
       (effects (font (size 1.27 1.27) italic) (justify left) hide)
     )
@@
       (effects (font (size 1.27 1.27)) (justify left))
     )
-    (property "Footprint" "Package_TO_SOT_THT:TO-92L_HandSolder" (id 2) (at 258.445 101.6 0)
+    (property "Footprint" "Package_TO_SOT_THT:TO-92_Inline_Wide" (id 2) (at 258.445 101.6 0)
       (effects (font (size 1.27 1.27) italic) (justify left) hide)
     )
@@
       (effects (font (size 1.27 1.27)) (justify left))
     )
-    (property "Footprint" "Package_TO_SOT_THT:TO-92L_HandSolder" (id 2) (at 304.165 101.6 0)
+    (property "Footprint" "Package_TO_SOT_THT:TO-92_Inline_Wide" (id 2) (at 304.165 101.6 0)
       (effects (font (size 1.27 1.27) italic) (justify left) hide)
     )
@@
       (effects (font (size 1.27 1.27)) (justify left))
     )
-    (property "Footprint" "Package_TO_SOT_THT:TO-92L_HandSolder" (id 2) (at 349.885 101.6 0)
+    (property "Footprint" "Package_TO_SOT_THT:TO-92_Inline_Wide" (id 2) (at 349.885 101.6 0)
       (effects (font (size 1.27 1.27) italic) (justify left) hide)
     )
@@
     )
     (path "/00000000-0000-0000-0000-000059826e5b"
-      (reference "Q1") (unit 1) (value "PN2222A") (footprint "Package_TO_SOT_THT:TO-92L_HandSolder")
+      (reference "Q1") (unit 1) (value "PN2222A") (footprint "Package_TO_SOT_THT:TO-92_Inline_Wide")
     )
     (path "/00000000-0000-0000-0000-00005a3b01a3"
-      (reference "Q2") (unit 1) (value "PN2222A") (footprint "Package_TO_SOT_THT:TO-92L_HandSolder")
+      (reference "Q2") (unit 1) (value "PN2222A") (footprint "Package_TO_SOT_THT:TO-92_Inline_Wide")
     )
     (path "/00000000-0000-0000-0000-00005a3b0732"
-      (reference "Q3") (unit 1) (value "PN2222A") (footprint "Package_TO_SOT_THT:TO-92L_HandSolder")
+      (reference "Q3") (unit 1) (value "PN2222A") (footprint "Package_TO_SOT_THT:TO-92_Inline_Wide")
     )
     (path "/00000000-0000-0000-0000-00005a3b081d"
-      (reference "Q4") (unit 1) (value "PN2222A") (footprint "Package_TO_SOT_THT:TO-92L_HandSolder")
+      (reference "Q4") (unit 1) (value "PN2222A") (footprint "Package_TO_SOT_THT:TO-92_Inline_Wide")
     )
     (path "/00000000-0000-0000-0000-00005a3b2528"
-      (reference "Q5") (unit 1) (value "PN2222A") (footprint "Package_TO_SOT_THT:TO-92L_HandSolder")
+      (reference "Q5") (unit 1) (value "PN2222A") (footprint "Package_TO_SOT_THT:TO-92_Inline_Wide")
     )
     (path "/00000000-0000-0000-0000-00005a3b2613"
-      (reference "Q6") (unit 1) (value "PN2222A") (footprint "Package_TO_SOT_THT:TO-92L_HandSolder")
+      (reference "Q6") (unit 1) (value "PN2222A") (footprint "Package_TO_SOT_THT:TO-92_Inline_Wide")
     )
     (path "/00000000-0000-0000-0000-00005a3b26fe"
-      (reference "Q7") (unit 1) (value "PN2222A") (footprint "Package_TO_SOT_THT:TO-92L_HandSolder")
+      (reference "Q7") (unit 1) (value "PN2222A") (footprint "Package_TO_SOT_THT:TO-92_Inline_Wide")
     )
     (path "/00000000-0000-0000-0000-00005a3b27e9"
-      (reference "Q8") (unit 1) (value "PN2222A") (footprint "Package_TO_SOT_THT:TO-92L_HandSolder")
+      (reference "Q8") (unit 1) (value "PN2222A") (footprint "Package_TO_SOT_THT:TO-92_Inline_Wide")
     )
     (path "/00000000-0000-0000-0000-0000598263cc"
@@
       (reference "R.D10") (unit 1) (value "270R") (footprint "Resistor_SMD:R_1206_3216Metric_Pad1.30x1.75mm_HandSolder")
     )
+    (path "/00000000-0000-0000-0000-00005db27a45"
+      (reference "R.R0") (unit 1) (value "2k") (footprint "Resistor_SMD:R_1206_3216Metric_Pad1.30x1.75mm_HandSolder")
+    )
+    (path "/00000000-0000-0000-0000-00005db2c8a5"
+      (reference "R.R1") (unit 1) (value "2k") (footprint "Resistor_SMD:R_1206_3216Metric_Pad1.30x1.75mm_HandSolder")
+    )
+    (path "/00000000-0000-0000-0000-00005db2ed55"
+      (reference "R.R2") (unit 1) (value "2k") (footprint "Resistor_SMD:R_1206_3216Metric_Pad1.30x1.75mm_HandSolder")
+    )
+    (path "/00000000-0000-0000-0000-00005db31435"
+      (reference "R.R3") (unit 1) (value "2k") (footprint "Resistor_SMD:R_1206_3216Metric_Pad1.30x1.75mm_HandSolder")
+    )
+    (path "/00000000-0000-0000-0000-00005db3377d"
+      (reference "R.R4") (unit 1) (value "2k") (footprint "Resistor_SMD:R_1206_3216Metric_Pad1.30x1.75mm_HandSolder")
+    )
+    (path "/00000000-0000-0000-0000-00005db35c7d"
+      (reference "R.R5") (unit 1) (value "2k") (footprint "Resistor_SMD:R_1206_3216Metric_Pad1.30x1.75mm_HandSolder")
+    )
     (path "/00000000-0000-0000-0000-00005982d566"
       (reference "R1") (unit 1) (value "1k") (footprint "Resistor_SMD:R_1206_3216Metric_Pad1.30x1.75mm_HandSolder")
@@
       (reference "R8") (unit 1) (value "1k") (footprint "Resistor_SMD:R_1206_3216Metric_Pad1.30x1.75mm_HandSolder")
     )
-    (path "/00000000-0000-0000-0000-00005db27a45"
-      (reference "R.R0") (unit 1) (value "2k") (footprint "Resistor_SMD:R_1206_3216Metric_Pad1.30x1.75mm_HandSolder")
-    )
-    (path "/00000000-0000-0000-0000-00005db2c8a5"
-      (reference "R.R1") (unit 1) (value "2k") (footprint "Resistor_SMD:R_1206_3216Metric_Pad1.30x1.75mm_HandSolder")
-    )
-    (path "/00000000-0000-0000-0000-00005db2ed55"
-      (reference "R.R2") (unit 1) (value "2k") (footprint "Resistor_SMD:R_1206_3216Metric_Pad1.30x1.75mm_HandSolder")
-    )
-    (path "/00000000-0000-0000-0000-00005db31435"
-      (reference "R.R3") (unit 1) (value "2k") (footprint "Resistor_SMD:R_1206_3216Metric_Pad1.30x1.75mm_HandSolder")
-    )
-    (path "/00000000-0000-0000-0000-00005db3377d"
-      (reference "R.R4") (unit 1) (value "2k") (footprint "Resistor_SMD:R_1206_3216Metric_Pad1.30x1.75mm_HandSolder")
-    )
-    (path "/00000000-0000-0000-0000-00005db35c7d"
-      (reference "R.R5") (unit 1) (value "2k") (footprint "Resistor_SMD:R_1206_3216Metric_Pad1.30x1.75mm_HandSolder")
-    )
     (path "/00000000-0000-0000-0000-0000598263bf"

Commit message: Add LCSC part numbers for the optocoupler schematics
Parts:
- Conn1: LCSC Part # (none) -> C692426
- Q1, Q2, Q3, Q4, Q5, Q6, Q7, Q8: LCSC Part # (none) -> C184875
- R.A0, R.A1, R.A10, R.A11, R.A2, R.A3, R.A4, R.A5, R.A6, R.A7, R.A8, R.A9, R.B0, R.B1, R.B10, R.B11, R.B12, R.B2, R.B3, R.B4, R.B5, R.B6, R.B7, R.B8, R.B9, R.C0, R.C1, R.C10, R.C11, R.C2, R.C3, R.C4, R.C5, R.C6, R.C7, R.C8, R.C9, R.D0, R.D1, R.D10, R.D2, R.D3, R.D4, R.D5, R.D6, R.D7, R.D8, R.D9: LCSC Part # (none) -> C229488
- R.R0, R.R1, R.R2, R.R3, R.R4, R.R5: LCSC Part # (none) -> C17944
- R1, R2, R3, R4, R5, R6, R7, R8: LCSC Part # (none) -> C4410
- U.A0, U.A1, U.A10, U.A11, U.A2, U.A3, U.A4, U.A5, U.A6, U.A7, U.A8, U.A9, U.B0, U.B1, U.B10, U.B11, U.B12, U.B2, U.B3, U.B4, U.B5, U.B6, U.B7, U.B8, U.B9, U.C0, U.C1, U.C10, U.C11, U.C2, U.C3, U.C4, U.C5, U.C6, U.C7, U.C8, U.C9, U.D0, U.D1, U.D10, U.D2, U.D3, U.D4, U.D5, U.D6, U.D7, U.D8, U.D9: LCSC Part # (none) -> C52833

Commit message: Replace rescued elements with proper / newer ones
Parts:
- Q1, Q2, Q3, Q4, Q5, Q6, Q7, Q8: symbol optocouplers-rescue:PN2222A-optocouplers-rescue -> Transistor_BJT:PN2222A
- R.A0, R.A1, R.A10, R.A11, R.A2, R.A3, R.A4, R.A5, R.A6, R.A7, R.A8, R.A9, R.B0, R.B1, R.B10, R.B11, R.B12, R.B2, R.B3, R.B4, R.B5, R.B6, R.B7, R.B8, R.B9, R.C0, R.C1, R.C10, R.C11, R.C2, R.C3, R.C4, R.C5, R.C6, R.C7, R.C8, R.C9, R.D0, R.D1, R.D10, R.D2, R.D3, R.D4, R.D5, R.D6, R.D7, R.D8, R.D9, R1, R2, R3, R4, R5, R6, R7, R8: symbol optocouplers-rescue:R-optocouplers-rescue -> Device:R
- U.A0, U.A1, U.A10, U.A11, U.A2, U.A3, U.A4, U.A5, U.A6, U.A7, U.A8, U.A9, U.B0, U.B1, U.B10, U.B11, U.B12, U.B2, U.B3, U.B4, U.B5, U.B6, U.B7, U.B8, U.B9, U.C0, U.C1, U.C10, U.C11, U.C2, U.C3, U.C4, U.C5, U.C6, U.C7, U.C8, U.C9, U.D0, U.D1, U.D10, U.D2, U.D3, U.D4, U.D5, U.D6, U.D7, U.D8, U.D9: symbol optocouplers-rescue:ITR9608-optocouplers-rescue -> Sensor_Proximity:ITR9608-F
Other:
- moved on the sheet: U.A0, U.A1, U.A10, U.A11, U.A2, U.A3, U.A4, U.A5, U.A6, U.A7, U.A8, U.A9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

Commit message: Use the new footprint for ITR9608
Parts:
- U.A0, U.A1, U.A10, U.A11, U.A2, U.A3, U.A4, U.A5, U.A6, U.A7, U.A8, U.A9, U.B0, U.B1, U.B10, U.B11, U.B12, U.B2, U.B3, U.B4, U.B5, U.B6, U.B7, U.B8, U.B9, U.C0, U.C1, U.C10, U.C11, U.C2, U.C3, U.C4, U.C5, U.C6, U.C7, U.C8, U.C9, U.D0, U.D1, U.D10, U.D2, U.D3, U.D4, U.D5, U.D6, U.D7, U.D8, U.D9: footprint ITR9608:ITR9608 -> OptoDevice:Everlight_ITR9608-F
