File: kicad/cherry-treble/cherry-treble.kicad_pcb (KiCad board)
At the start: 2 copper layers, 299 x 129 mm, 103 parts

Commit message: Update cherry treble PCB
Parts:
- added ?: , , F.Cu at (25.0, 102.0)
- added ?: , , F.Cu at (280.0, 102.0)
- added ?: , , F.Cu at (280.0, 5.00)
- added ?: , , F.Cu at (25.0, 5.00)
- R0, R1, R2, R3, R4, R5: moved to B.Cu
- moved R0 190.9 mm to (46.5, 64.8)
- moved R1 181.8 mm to (66.5, 64.8)
- moved R2 172.7 mm to (86.5, 64.8)
- moved R3 163.8 mm to (106.5, 64.8)
- moved R4 154.9 mm to (126.5, 64.8)
- moved R5 146.3 mm to (146.6, 64.8)
- moved Conn1 138.2 mm to (84.8, 10.8)
Routing:
- net arduino_A1: track 149.8 -> 378.1 mm, vias 0 -> 2
- net arduino_A5: track 159.9 -> 386.5 mm, vias 0 -> 3
- net arduino_A0: track 179.8 -> 391.0 mm
- net arduino_A4: track 179.8 -> 387.8 mm, vias 0 -> 3
- net arduino_A3: track 179.8 -> 382.1 mm, vias 0 -> 2
- net arduino_A2: track 179.7 -> 370.8 mm, vias 0 -> 2
- net arduino_D6: track 100.0 -> 251.5 mm
- net arduino_D5: track 100.0 -> 241.9 mm
- net arduino_D8: track 100.4 -> 219.5 mm
- net arduino_D7: track 102.3 -> 218.9 mm, vias 0 -> 1
- net arduino_D9: track 100.0 -> 198.7 mm, vias 0 -> 1
- net arduino_D10: track 100.3 -> 193.3 mm
- net arduino_D12: track 144.9 -> 220.3 mm
- net arduino_D11: track 100.1 -> 133.4 mm
- net GND: vias 0 -> 3
- added copper zone on B.Cu, net GND
- added copper zone on F.Cu, net GND
Other:
- board size 299 x 129 mm -> 265 x 107 mm
- board text added: "(Aug 2022)"
- board text added: "Midiatonerca 1.0"
- board text added: "Proudly presented by Mojca & Vincent"

Commit message: Move connector closer to the keys on cherry treble
Almost enforce the clearance
Parts:
- moved Conn1 5.34 mm to (88.0, 15.0)
Routing:
- net arduino_D12: track 220.3 -> 206.1 mm
- net arduino_D10: track 193.3 -> 181.8 mm
- net arduino_D6: track 251.5 -> 241.0 mm
- net arduino_D8: track 219.5 -> 209.1 mm
- net arduino_A4: track 387.8 -> 383.0 mm
- net arduino_D7: track 218.9 -> 214.3 mm
- net arduino_D9: track 198.7 -> 194.4 mm
- net arduino_A5: track 386.5 -> 382.2 mm
- net arduino_A1: track 378.1 -> 374.1 mm
- net arduino_A2: track 370.8 -> 366.9 mm
- net arduino_D11: track 133.4 -> 129.9 mm
- net arduino_A3: track 382.1 -> 379.0 mm
- net arduino_A0: track 391.0 -> 392.5 mm
- net arduino_D5: track 241.9 -> 240.5 mm
- net GND: vias 3 -> 5

Commit message: Move elements of the cherry treble PCB
Parts:
- moved ? 20.1 mm to (5.00, 100.0)
- moved ? 20.0 mm to (5.00, 5.00)
- moved Conn1 15.8 mm to (73.0, 10.0)
- moved D.A0 15.8 mm to (30.0, 81.0)
- moved D.A1 15.8 mm to (50.0, 81.0)
- moved D.A10 15.8 mm to (230.0, 81.0)
- moved D.A11 15.8 mm to (250.0, 81.0)
- moved D.A2 15.8 mm to (70.0, 81.0)
- moved D.A3 15.8 mm to (90.0, 81.0)
- moved D.A4 15.8 mm to (110.0, 81.0)
- moved D.A5 15.8 mm to (130.0, 81.0)
- moved D.A6 15.8 mm to (150.0, 81.0)
- moved D.A7 15.8 mm to (170.0, 81.0)
- moved D.A8 15.8 mm to (190.0, 81.0)
- moved D.A9 15.8 mm to (210.0, 81.0)
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Other:
- board size 265 x 107 mm -> 275 x 105 mm

Commit message: Potentially finished cherry treble pcb
Parts:
- removed the ? at (5.00, 100.0)
- added ?: , , F.Cu at (217.0, 5.00)
- added ?: , , F.Cu at (111.0, 105.0)
- added ?: , , F.Cu at (58.0, 105.0)
- added ?: , , F.Cu at (164.0, 5.00)
- added ?: , , F.Cu at (58.0, 5.00)
- added ?: , , F.Cu at (270.0, 55.0)
- added ?: , , F.Cu at (217.0, 105.0)
- added ?: , , F.Cu at (164.0, 105.0)
- added ?: , , F.Cu at (5.00, 55.0)
- added ?: , , F.Cu at (5.00, 105.0)
- added ?: , , F.Cu at (111.0, 5.00)
- moved ? 5.00 mm to (270.0, 105.0)
- moved Conn1 3.68 mm to (69.8, 11.8)
Routing:
- net arduino_A0: track 392.5 -> 386.0 mm
- net arduino_D7: track 214.3 -> 210.3 mm
- net arduino_D5: track 240.5 -> 236.5 mm
- net arduino_D9: track 194.4 -> 190.4 mm
- net arduino_A1: track 374.1 -> 370.3 mm
- net arduino_D8: track 209.1 -> 211.6 mm
- net arduino_D12: track 206.1 -> 208.6 mm
- net arduino_D10: track 181.8 -> 184.3 mm
- net arduino_D11: track 129.9 -> 127.6 mm
- net arduino_D6: track 241.0 -> 243.0 mm
- net arduino_A5: track 382.2 -> 383.9 mm
- net arduino_A2: track 366.9 -> 365.7 mm
- net arduino_A4: track 383.0 -> 381.8 mm
- net GND: vias 5 -> 43
Other:
- board size 275 x 105 mm -> 275 x 110 mm
- rule pad_to_mask_clearance: 0.051 -> 0

Commit message: shrink cherry treble pcb by 2 mm on each side
Parts:
- moved ? 1.00 mm to (6.00, 5.00)
- moved ? 1.00 mm to (269.0, 55.0)
- moved ? 1.00 mm to (269.0, 105.0)
- moved ? 1.00 mm to (6.00, 55.0)
- moved ? 1.00 mm to (6.00, 105.0)
- moved ? 1.00 mm to (269.0, 5.00)
Other:
- board size 275 x 110 mm -> 271 x 110 mm
Changed lines of the file:
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@@
   )
   (footprint "" (layer "F.Cu")
-    (at 270 55)
+    (at 269 55)
     (fp_text reference "" (at 0 0) (layer "F.SilkS")
       (effects (font (size 1.27 1.27) (thickness 0.15)))
@@
   )
   (footprint "" (layer "F.Cu")
-    (at 270 105)
+    (at 269 105)
     (fp_text reference "" (at 0 0) (layer "F.SilkS")
       (effects (font (size 1.27 1.27) (thickness 0.15)))
@@
   )
   (footprint "" (layer "F.Cu")
-    (at 5 55)
+    (at 6 55)
     (fp_text reference "" (at 0 0) (layer "F.SilkS")
       (effects (font (size 1.27 1.27) (thickness 0.15)))
@@
   )
   (footprint "" (layer "F.Cu")
-    (at 5 105)
+    (at 6 105)
     (fp_text reference "" (at 0 0) (layer "F.SilkS")
       (effects (font (size 1.27 1.27) (thickness 0.15)))
@@
   )
   (footprint "" (layer "F.Cu")
-    (at 270 5)
+    (at 269 5)
     (fp_text reference "" (at 0 0) (layer "F.SilkS")
       (effects (font (size 1.27 1.27) (thickness 0.15)))
@@
   )
   (footprint "" (layer "F.Cu")
-    (at 5 5)
+    (at 6 5)
     (fp_text reference "" (at 0 0) (layer "F.SilkS")
       (effects (font (size 1.27 1.27) (thickness 0.15)))
@@
     )
   )
-  (gr_rect (start 0 0) (end 275 110) (layer "Edge.Cuts") (width 0.1) (fill none))
+  (gr_rect (start 2 0) (end 273 110) (layer "Edge.Cuts") (width 0.1) (fill none))
   (gr_text "Proudly presented by Mojca & Vincent" (at 262 11) (layer "B.SilkS")
     (effects (font (size 2 1.8) (thickness 0.2)) (justify left mirror))
@@
     (connect_pads (clearance 0.508))
     (min_thickness 0.254) (filled_areas_thickness no)
-    (fill yes (thermal_gap 0.508) (thermal_bridge_width 0.508))
+    (fill (thermal_gap 0.508) (thermal_bridge_width 0.508))
     (polygon
       (pts
-        (xy 275 110)
-        (xy 0 110)
-        (xy 0 0)
-        (xy 275 0)
+        (xy 273 110)
+        (xy 2 110)
+        (xy 2 0)
+        (xy 273 0)
       )
     )

Commit message: Shrink kicad treble, fix interline spacing
Parts:
- moved ? 6.00 mm to (217.0, 11.0)
- moved ? 6.00 mm to (6.00, 11.0)
- moved ? 6.00 mm to (164.0, 11.0)
- moved ? 6.00 mm to (58.0, 11.0)
- moved ? 6.00 mm to (111.0, 11.0)
- moved ? 6.00 mm to (269.0, 11.0)
- moved Conn1 5.40 mm to (69.8, 17.2)
- moved D.D0 5.40 mm to (40.0, 26.4)
- moved D.D1 5.40 mm to (60.0, 26.4)
- moved D.D10 5.40 mm to (240.0, 26.4)
- moved D.D2 5.40 mm to (80.0, 26.4)
- moved D.D3 5.40 mm to (100.0, 26.4)
- moved D.D4 5.40 mm to (120.0, 26.4)
- moved D.D5 5.40 mm to (140.0, 26.4)
- moved D.D6 5.40 mm to (160.0, 26.4)
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Routing:
- net arduino_A1: track 370.3 -> 354.0 mm
- net arduino_A0: track 386.0 -> 369.8 mm
- net arduino_A3: track 379.0 -> 362.8 mm
- net arduino_A2: track 365.7 -> 349.4 mm
- net arduino_A4: track 381.8 -> 365.6 mm
- net arduino_A5: track 383.9 -> 370.2 mm
- net arduino_D6: track 243.0 -> 234.9 mm
- net arduino_D5: track 236.5 -> 228.4 mm
- net arduino_D12: track 208.6 -> 203.2 mm
- net arduino_D7: track 210.3 -> 204.9 mm
- net arduino_D8: track 211.6 -> 206.2 mm
- net arduino_D9: track 190.4 -> 187.7 mm
- net arduino_D10: track 184.3 -> 181.6 mm
Other:
- board size 271 x 110 mm -> 271 x 95 mm

Commit message: Further dimension adjustments to cherry treble to fit into the box
Parts:
- moved ? 3.06 mm to (58.6, 97.0)
- moved ? 3.06 mm to (216.4, 97.0)
- moved ? 3.01 mm to (111.2, 97.0)
- moved ? 3.01 mm to (163.8, 97.0)
- moved ? 3.00 mm to (269.0, 97.0)
- moved ? 3.00 mm to (6.00, 97.0)
- moved ? 1.00 mm to (269.0, 54.0)
- moved ? 1.00 mm to (6.00, 54.0)
- moved ? 0.60 mm to (58.6, 11.0)
- moved ? 0.60 mm to (216.4, 11.0)
- moved ? 0.20 mm to (111.2, 11.0)
- moved ? 0.20 mm to (163.8, 11.0)
Routing:
- net arduino_A4: track 365.6 -> 330.6 mm, vias 3 -> 2
- net arduino_A5: track 370.2 -> 350.5 mm, vias 3 -> 2
- net arduino_A3: track 362.8 -> 344.3 mm, vias 2 -> 1
Other:
- board size 271 x 95 mm -> 271 x 92.5 mm
