File: kicad/cherry-treble/cherry-treble.kicad_pcb (KiCad board)
At the start: 2 copper layers, 271 x 92.5 mm, 117 parts

Commit message: Rename diodes on the PCB (probably not needed, might be reverted)
Parts:
- D.A0, D.A1, D.A10, D.A11, D.A2, D.A3, D.A4, D.A5, D.A6, D.A7, D.A8, D.A9, D.B0, D.B1, D.B10, D.B11, D.B12, D.B2, D.B3, D.B4, D.B5, D.B6, D.B7, D.B8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: value DIODE -> 1N4148WS
