File: kicad/cherry-treble/cherry-treble.kicad_pcb (KiCad board)
At the start: 2 copper layers, 271 x 92.5 mm, 117 parts

Commit message: Update diodes from schematic and fix polarity on cherry treble pcb
Parts:
- D.A0, D.A1, D.A10, D.A11, D.A2, D.A3, D.A4, D.A5, D.A6, D.A7, D.A8, D.A9, D.B0, D.B1, D.B10, D.B11, D.B12, D.B2, D.B3, D.B4, D.B5, D.B6, D.B7, D.B8, D.B9, D.C0, D.C1, D.C10, D.C11, D.C2, D.C3, D.C4, D.C5, D.C6, D.C7, D.C8, D.C9, D.D0, D.D1, D.D10, D.D2, D.D3, D.D4, D.D5, D.D6, D.D7, D.D8, D.D9: value 1N4148WS -> 1N5819WS
- turned D.A0 to -90 degrees
- turned D.A1 to -90 degrees
- turned D.A10 to -90 degrees
- turned D.A11 to -90 degrees
- turned D.A2 to -90 degrees
- turned D.A3 to -90 degrees
- turned D.A4 to -90 degrees
- turned D.A5 to -90 degrees
- turned D.A6 to -90 degrees
- turned D.A7 to -90 degrees
- turned D.A8 to -90 degrees
- turned D.A9 to -90 degrees
- turned D.B0 to -90 degrees
- turned D.B1 to -90 degrees
- turned D.B10 to -90 degrees
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Connections:
- D.A0 pad 1: Net-(D.A0-Pad1) -> arduino_A0
- D.A0 pad 2: arduino_A0 -> Net-(D.A0-Pad2)
- D.A1 pad 1: Net-(D.A1-Pad1) -> arduino_A1
- D.A1 pad 2: arduino_A1 -> Net-(D.A1-Pad2)
- D.A10 pad 1: Net-(D.A10-Pad1) -> arduino_A4
- D.A10 pad 2: arduino_A4 -> Net-(D.A10-Pad2)
- D.A11 pad 1: Net-(D.A11-Pad1) -> arduino_A5
- D.A11 pad 2: arduino_A5 -> Net-(D.A11-Pad2)
- D.A2 pad 1: Net-(D.A2-Pad1) -> arduino_A2
- D.A2 pad 2: arduino_A2 -> Net-(D.A2-Pad2)
- D.A3 pad 1: Net-(D.A3-Pad1) -> arduino_A3
- D.A3 pad 2: arduino_A3 -> Net-(D.A3-Pad2)
- D.A4 pad 1: Net-(D.A4-Pad1) -> arduino_A4
- D.A4 pad 2: arduino_A4 -> Net-(D.A4-Pad2)
- D.A5 pad 1: Net-(D.A5-Pad1) -> arduino_A5
- D.A5 pad 2: arduino_A5 -> Net-(D.A5-Pad2)
- D.A6 pad 1: Net-(D.A6-Pad1) -> arduino_A0
- D.A6 pad 2: arduino_A0 -> Net-(D.A6-Pad2)
- D.A7 pad 1: Net-(D.A7-Pad1) -> arduino_A1
- D.A7 pad 2: arduino_A1 -> Net-(D.A7-Pad2)
- D.A8 pad 1: Net-(D.A8-Pad1) -> arduino_A2
- D.A8 pad 2: arduino_A2 -> Net-(D.A8-Pad2)
- D.A9 pad 1: Net-(D.A9-Pad1) -> arduino_A3
- D.A9 pad 2: arduino_A3 -> Net-(D.A9-Pad2)
- D.B0 pad 1: Net-(D.B0-Pad1) -> arduino_A0
- D.B0 pad 2: arduino_A0 -> Net-(D.B0-Pad2)
- D.B1 pad 1: Net-(D.B1-Pad1) -> arduino_A1
- D.B1 pad 2: arduino_A1 -> Net-(D.B1-Pad2)
- D.B10 pad 1: Net-(D.B10-Pad1) -> arduino_A4
- D.B10 pad 2: arduino_A4 -> Net-(D.B10-Pad2)
- D.B11 pad 1: Net-(D.B11-Pad1) -> arduino_A5
- D.B11 pad 2: arduino_A5 -> Net-(D.B11-Pad2)
- D.B12 pad 1: Net-(D.B12-Pad1) -> arduino_A5
- D.B12 pad 2: arduino_A5 -> Net-(D.B12-Pad2)
- D.B2 pad 1: Net-(D.B2-Pad1) -> arduino_A2
- D.B2 pad 2: arduino_A2 -> Net-(D.B2-Pad2)
- D.B3 pad 1: Net-(D.B3-Pad1) -> arduino_A3
- D.B3 pad 2: arduino_A3 -> Net-(D.B3-Pad2)
- D.B4 pad 1: Net-(D.B4-Pad1) -> arduino_A4
- D.B4 pad 2: arduino_A4 -> Net-(D.B4-Pad2)
- D.B5 pad 1: Net-(D.B5-Pad1) -> arduino_A5
- D.B5 pad 2: arduino_A5 -> Net-(D.B5-Pad2)
- D.B6 pad 1: Net-(D.B6-Pad1) -> arduino_A0
- D.B6 pad 2: arduino_A0 -> Net-(D.B6-Pad2)
- D.B7 pad 1: Net-(D.B7-Pad1) -> arduino_A1
- D.B7 pad 2: arduino_A1 -> Net-(D.B7-Pad2)
- D.B8 pad 1: Net-(D.B8-Pad1) -> arduino_A2
- D.B8 pad 2: arduino_A2 -> Net-(D.B8-Pad2)
- D.B9 pad 1: Net-(D.B9-Pad1) -> arduino_A3
- D.B9 pad 2: arduino_A3 -> Net-(D.B9-Pad2)
- D.C0 pad 1: Net-(D.C0-Pad1) -> arduino_A0
- D.C0 pad 2: arduino_A0 -> Net-(D.C0-Pad2)
- D.C1 pad 1: Net-(D.C1-Pad1) -> arduino_A1
- D.C1 pad 2: arduino_A1 -> Net-(D.C1-Pad2)
- D.C10 pad 1: Net-(D.C10-Pad1) -> arduino_A4
- D.C10 pad 2: arduino_A4 -> Net-(D.C10-Pad2)
- D.C11 pad 1: Net-(D.C11-Pad1) -> arduino_A5
- D.C11 pad 2: arduino_A5 -> Net-(D.C11-Pad2)
- D.C2 pad 1: Net-(D.C2-Pad1) -> arduino_A2
- D.C2 pad 2: arduino_A2 -> Net-(D.C2-Pad2)
- D.C3 pad 1: Net-(D.C3-Pad1) -> arduino_A3
- D.C3 pad 2: arduino_A3 -> Net-(D.C3-Pad2)
- D.C4 pad 1: Net-(D.C4-Pad1) -> arduino_A4
- D.C4 pad 2: arduino_A4 -> Net-(D.C4-Pad2)
- D.C5 pad 1: Net-(D.C5-Pad1) -> arduino_A5
- D.C5 pad 2: arduino_A5 -> Net-(D.C5-Pad2)
- D.C6 pad 1: Net-(D.C6-Pad1) -> arduino_A0
- D.C6 pad 2: arduino_A0 -> Net-(D.C6-Pad2)
- D.C7 pad 1: Net-(D.C7-Pad1) -> arduino_A1
- D.C7 pad 2: arduino_A1 -> Net-(D.C7-Pad2)
- D.C8 pad 1: Net-(D.C8-Pad1) -> arduino_A2
- D.C8 pad 2: arduino_A2 -> Net-(D.C8-Pad2)
- D.C9 pad 1: Net-(D.C9-Pad1) -> arduino_A3
- D.C9 pad 2: arduino_A3 -> Net-(D.C9-Pad2)
- D.D0 pad 1: Net-(D.D0-Pad1) -> arduino_A0
- D.D0 pad 2: arduino_A0 -> Net-(D.D0-Pad2)
- D.D1 pad 1: Net-(D.D1-Pad1) -> arduino_A1
- D.D1 pad 2: arduino_A1 -> Net-(D.D1-Pad2)
- D.D10 pad 1: Net-(D.D10-Pad1) -> arduino_A4
- D.D10 pad 2: arduino_A4 -> Net-(D.D10-Pad2)
- D.D2 pad 1: Net-(D.D2-Pad1) -> arduino_A2
- D.D2 pad 2: arduino_A2 -> Net-(D.D2-Pad2)
- D.D3 pad 1: Net-(D.D3-Pad1) -> arduino_A3
- D.D3 pad 2: arduino_A3 -> Net-(D.D3-Pad2)
- D.D4 pad 1: Net-(D.D4-Pad1) -> arduino_A4
- D.D4 pad 2: arduino_A4 -> Net-(D.D4-Pad2)
- D.D5 pad 1: Net-(D.D5-Pad1) -> arduino_A5
- D.D5 pad 2: arduino_A5 -> Net-(D.D5-Pad2)
- D.D6 pad 1: Net-(D.D6-Pad1) -> arduino_A0
- D.D6 pad 2: arduino_A0 -> Net-(D.D6-Pad2)
- D.D7 pad 1: Net-(D.D7-Pad1) -> arduino_A1
- D.D7 pad 2: arduino_A1 -> Net-(D.D7-Pad2)
- D.D8 pad 1: Net-(D.D8-Pad1) -> arduino_A2
- D.D8 pad 2: arduino_A2 -> Net-(D.D8-Pad2)
- D.D9 pad 1: Net-(D.D9-Pad1) -> arduino_A3
- D.D9 pad 2: arduino_A3 -> Net-(D.D9-Pad2)
- SW.A0 pad 1: Net-(D.A0-Pad1) -> Net-(D.A0-Pad2)
- SW.A1 pad 1: Net-(D.A1-Pad1) -> Net-(D.A1-Pad2)
- SW.A10 pad 1: Net-(D.A10-Pad1) -> Net-(D.A10-Pad2)
- SW.A11 pad 1: Net-(D.A11-Pad1) -> Net-(D.A11-Pad2)
- SW.A2 pad 1: Net-(D.A2-Pad1) -> Net-(D.A2-Pad2)
- SW.A3 pad 1: Net-(D.A3-Pad1) -> Net-(D.A3-Pad2)
- SW.A4 pad 1: Net-(D.A4-Pad1) -> Net-(D.A4-Pad2)
- SW.A5 pad 1: Net-(D.A5-Pad1) -> Net-(D.A5-Pad2)
- SW.A6 pad 1: Net-(D.A6-Pad1) -> Net-(D.A6-Pad2)
- SW.A7 pad 1: Net-(D.A7-Pad1) -> Net-(D.A7-Pad2)
- SW.A8 pad 1: Net-(D.A8-Pad1) -> Net-(D.A8-Pad2)
- SW.A9 pad 1: Net-(D.A9-Pad1) -> Net-(D.A9-Pad2)
- SW.B0 pad 1: Net-(D.B0-Pad1) -> Net-(D.B0-Pad2)
- SW.B1 pad 1: Net-(D.B1-Pad1) -> Net-(D.B1-Pad2)
- SW.B10 pad 1: Net-(D.B10-Pad1) -> Net-(D.B10-Pad2)
- SW.B11 pad 1: Net-(D.B11-Pad1) -> Net-(D.B11-Pad2)
- SW.B12 pad 1: Net-(D.B12-Pad1) -> Net-(D.B12-Pad2)
- SW.B2 pad 1: Net-(D.B2-Pad1) -> Net-(D.B2-Pad2)
- SW.B3 pad 1: Net-(D.B3-Pad1) -> Net-(D.B3-Pad2)
- SW.B4 pad 1: Net-(D.B4-Pad1) -> Net-(D.B4-Pad2)
- SW.B5 pad 1: Net-(D.B5-Pad1) -> Net-(D.B5-Pad2)
- SW.B6 pad 1: Net-(D.B6-Pad1) -> Net-(D.B6-Pad2)
- SW.B7 pad 1: Net-(D.B7-Pad1) -> Net-(D.B7-Pad2)
- SW.B8 pad 1: Net-(D.B8-Pad1) -> Net-(D.B8-Pad2)
- SW.B9 pad 1: Net-(D.B9-Pad1) -> Net-(D.B9-Pad2)
- SW.C0 pad 1: Net-(D.C0-Pad1) -> Net-(D.C0-Pad2)
- SW.C1 pad 1: Net-(D.C1-Pad1) -> Net-(D.C1-Pad2)
- SW.C10 pad 1: Net-(D.C10-Pad1) -> Net-(D.C10-Pad2)
- SW.C11 pad 1: Net-(D.C11-Pad1) -> Net-(D.C11-Pad2)
- SW.C2 pad 1: Net-(D.C2-Pad1) -> Net-(D.C2-Pad2)
- SW.C3 pad 1: Net-(D.C3-Pad1) -> Net-(D.C3-Pad2)
- SW.C4 pad 1: Net-(D.C4-Pad1) -> Net-(D.C4-Pad2)
- SW.C5 pad 1: Net-(D.C5-Pad1) -> Net-(D.C5-Pad2)
- SW.C6 pad 1: Net-(D.C6-Pad1) -> Net-(D.C6-Pad2)
- SW.C7 pad 1: Net-(D.C7-Pad1) -> Net-(D.C7-Pad2)
- SW.C8 pad 1: Net-(D.C8-Pad1) -> Net-(D.C8-Pad2)
- SW.C9 pad 1: Net-(D.C9-Pad1) -> Net-(D.C9-Pad2)
- SW.D0 pad 1: Net-(D.D0-Pad1) -> Net-(D.D0-Pad2)
- SW.D1 pad 1: Net-(D.D1-Pad1) -> Net-(D.D1-Pad2)
- SW.D10 pad 1: Net-(D.D10-Pad1) -> Net-(D.D10-Pad2)
- SW.D2 pad 1: Net-(D.D2-Pad1) -> Net-(D.D2-Pad2)
- SW.D3 pad 1: Net-(D.D3-Pad1) -> Net-(D.D3-Pad2)
- SW.D4 pad 1: Net-(D.D4-Pad1) -> Net-(D.D4-Pad2)
- SW.D5 pad 1: Net-(D.D5-Pad1) -> Net-(D.D5-Pad2)
- SW.D6 pad 1: Net-(D.D6-Pad1) -> Net-(D.D6-Pad2)
- SW.D7 pad 1: Net-(D.D7-Pad1) -> Net-(D.D7-Pad2)
- SW.D8 pad 1: Net-(D.D8-Pad1) -> Net-(D.D8-Pad2)
- SW.D9 pad 1: Net-(D.D9-Pad1) -> Net-(D.D9-Pad2)
Routing:
- net Net-(D.D9-Pad2): track 0.00 -> 2.75 mm
- net Net-(D.D9-Pad1): track 2.75 -> 0.00 mm
- net Net-(D.D8-Pad2): track 0.00 -> 2.75 mm
- net Net-(D.D8-Pad1): track 2.75 -> 0.00 mm
- net Net-(D.D7-Pad2): track 0.00 -> 2.75 mm
- net Net-(D.D7-Pad1): track 2.75 -> 0.00 mm
- net Net-(D.D6-Pad2): track 0.00 -> 2.75 mm
- net Net-(D.D6-Pad1): track 2.75 -> 0.00 mm
- net Net-(D.D5-Pad2): track 0.00 -> 2.75 mm
- net Net-(D.D5-Pad1): track 2.75 -> 0.00 mm
- net Net-(D.D4-Pad2): track 0.00 -> 2.75 mm
- net Net-(D.D4-Pad1): track 2.75 -> 0.00 mm
- net Net-(D.D3-Pad2): track 0.00 -> 2.75 mm
- net Net-(D.D3-Pad1): track 2.75 -> 0.00 mm
- net Net-(D.D2-Pad2): track 0.00 -> 2.75 mm
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
Commit message: Avoid 90 degree corners in cherry treble pcb
Parts:
- moved R0 2.55 mm to (31.6, 62.3)
- moved R1 2.55 mm to (51.5, 62.3)
- moved R2 2.55 mm to (71.5, 62.3)
- moved R3 2.55 mm to (91.5, 62.3)
- moved R4 2.55 mm to (111.5, 62.3)
- moved R5 2.55 mm to (131.6, 62.3)
Routing:
- net arduino_A0: track 369.8 -> 361.2 mm
- net arduino_A1: track 354.0 -> 345.5 mm
- net arduino_A2: track 349.4 -> 342.4 mm
- net arduino_A4: track 330.6 -> 324.3 mm
- net arduino_A3: track 344.3 -> 338.6 mm
- net arduino_A5: track 350.5 -> 346.2 mm

Commit message: Add kicad & osh symbols to cherry treble pcb
Parts:
- added REF**: OSHW-Logo2_14.6x12mm_SilkScreen, Symbol:OSHW-Logo2_14.6x12mm_SilkScreen, F.Cu at (258.0, 33.0)
- added REF**: KiCad-Logo2_5mm_SilkScreen, Symbol:KiCad-Logo2_5mm_SilkScreen, F.Cu at (19.0, 36.0)
- added REF**: KiCad-Logo2_5mm_SilkScreen, Symbol:KiCad-Logo2_5mm_SilkScreen, B.Cu at (19.0, 36.0)
- added REF**: OSHW-Logo2_14.6x12mm_SilkScreen, Symbol:OSHW-Logo2_14.6x12mm_SilkScreen, B.Cu at (258.0, 33.0)
