File: kicad/cherry-treble/cherry-treble.kicad_sch (KiCad schematic)
At the start: 103 parts

Commit message: Fix part number for the schottky diodes
Parts:
- D.A0, D.A1, D.A10, D.A11, D.A2, D.A3, D.A4, D.A5, D.A6, D.A7, D.A8, D.A9, D.B0, D.B1, D.B10, D.B11, D.B12, D.B2, D.B3, D.B4, D.B5, D.B6, D.B7, D.B8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: LCSC Part # C2128 -> C191023
