File: kicad/arduino-plate/arduino-plate.kicad_sch (KiCad schematic)
At the start: 6 parts

Commit message: Updates to arduino
Parts:
- renumbered J.3 to J.Pres.1, J.2 to J.VM.1
Changed lines of the file:
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@@
   (no_connect (at 107.95 54.61))
   (no_connect (at 45.72 69.85))
+  (no_connect (at 30.48 62.23))
   (no_connect (at 107.95 52.07))
   (no_connect (at 107.95 49.53))
@@
   (no_connect (at 45.72 19.05))
   (no_connect (at 55.88 29.21))
-  (no_connect (at 30.48 62.23))
   (no_connect (at 30.48 31.75))
   (no_connect (at 30.48 29.21))
@@
   (symbol (lib_id "Connector:Conn_01x03_Male") (at 74.93 83.82 270) (unit 1)
     (in_bom yes) (on_board yes) (fields_autoplaced)
-    (property "Reference" "J.3" (id 0) (at 74.93 78.74 90))
+    (property "Reference" "J.Pres.1" (id 0) (at 74.93 78.74 90))
     (property "Value" "Conn_01x03_Male" (id 1) (at 74.93 81.28 90))
     (property "Footprint" "Connector_Molex:Molex_KK-254_AE-6410-03A_1x03_P2.54mm_Vertical" (id 2) (at 74.93 83.82 0)
@@
   (symbol (lib_id "Connector:Conn_01x02_Male") (at 36.83 83.82 270) (unit 1)
     (in_bom yes) (on_board yes) (fields_autoplaced)
-    (property "Reference" "J.2" (id 0) (at 38.1 83.1849 90)
+    (property "Reference" "J.VM.1" (id 0) (at 38.1 83.1849 90)
       (effects (font (size 1.27 1.27)) (justify left))
     )
@@
       (reference "J.1") (unit 1) (value "Conn_02x13_Odd_Even") (footprint "Connector_IDC:IDC-Header_2x13_P2.54mm_Vertical")
     )
+    (path "/28de4405-1021-43ed-988e-12cdf1abb148"
+      (reference "J.Pres.1") (unit 1) (value "Conn_01x03_Male") (footprint "Connector_Molex:Molex_KK-254_AE-6410-03A_1x03_P2.54mm_Vertical")
+    )
     (path "/b8d379d6-3088-4109-ae1f-421f48a1b55f"
-      (reference "J.2") (unit 1) (value "Conn_01x02_Male") (footprint "Connector_Molex:Molex_KK-254_AE-6410-02A_1x02_P2.54mm_Vertical")
-    )
-    (path "/28de4405-1021-43ed-988e-12cdf1abb148"
-      (reference "J.3") (unit 1) (value "Conn_01x03_Male") (footprint "Connector_Molex:Molex_KK-254_AE-6410-03A_1x03_P2.54mm_Vertical")
+      (reference "J.VM.1") (unit 1) (value "Conn_01x02_Male") (footprint "Connector_Molex:Molex_KK-254_AE-6410-02A_1x02_P2.54mm_Vertical")
     )
     (path "/e466fdd1-256e-40af-a34f-fa99f58d4c57"
