File: kicad/led-strip/led-strip.kicad_pcb (KiCad board)
At the start: 2 copper layers, 257 x 8 mm, 29 parts, among them J1 Conn_01x03, J2 Conn_01x03, J3 Conn_01x03, J4 Conn_01x03

Commit message: led strip pcb: improve pad connections at the end, positive polarity zone ipd.
Parts:
- moved J1 0.50 mm to (24.5, 49.0)
- moved J4 0.50 mm to (275.5, 49.0)
Routing:
- net +5V: track 674.3 -> 421.5 mm
- net GND: track 90.8 -> 251.6 mm, vias 15 -> 14
- net Net-(D13-Pad2): track 3.82 -> 3.32 mm
- net Net-(D1-Pad4): track 4.61 -> 4.11 mm
- added copper zone on B.Cu, net +5V
- added copper zone on F.Cu, net +5V
