File: kicad/rpi-audio-hat/rpi-audio-hat.kicad_pcb (KiCad board)
At the start: 4 copper layers, 65 x 56 mm, 32 parts, among them J1 Raspberry_Pi_2_3, J2 Conn_Volume_Slider, J3 Screw_Terminal_01x02, J4 Screw_Terminal_01x02, J5 Screw_Terminal_01x02, SW1 SW_SPDT, U1 PCM5102_breakout, U2 PAM8302A_Adafruit_Board, U3 SLM6800, U4 PCM5102A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

Commit message: Save PCB
Parts:
- added C16: 1uF, Capacitor_SMD:C_0603_1608Metric, F.Cu at (112.9, 78.6)
- added C17: 1uF, Capacitor_SMD:C_0603_1608Metric, F.Cu at (112.9, 81.1)
- added C18: 10uF, Capacitor_SMD:C_0603_1608Metric, F.Cu at (112.9, 83.6)
- added C19: 100nF, Capacitor_SMD:C_0603_1608Metric, F.Cu at (127.2, 71.2)
- added C20: 100nF, Capacitor_SMD:C_0603_1608Metric, F.Cu at (107.4, 78.2)
- added C21: 22uF, Capacitor_SMD:C_1206_3216Metric, F.Cu at (102.6, 78.6)
- added C22: 22uF, Capacitor_SMD:C_1206_3216Metric, F.Cu at (102.6, 82.0)
- added C23: 22pF, Capacitor_SMD:C_0603_1608Metric, F.Cu at (107.4, 80.7)
- added C24: 22uF, Capacitor_SMD:C_1206_3216Metric, F.Cu at (102.6, 85.3)
- added C25: 22uF, Capacitor_SMD:C_1206_3216Metric, F.Cu at (102.6, 88.7)
- added C26: 100nF, Capacitor_SMD:C_0603_1608Metric, F.Cu at (107.4, 83.2)
- added C27: 22pF, Capacitor_SMD:C_0603_1608Metric, F.Cu at (107.4, 85.8)
- added C28: 22uF, Capacitor_SMD:C_1206_3216Metric, F.Cu at (102.6, 92.0)
- added C29: 22uF, Capacitor_SMD:C_1206_3216Metric, F.Cu at (102.6, 95.4)
- added C3: 100nF, Capacitor_SMD:C_0603_1608Metric, F.Cu at (127.2, 68.7)
- added C30: 22uF, Capacitor_SMD:C_1206_3216Metric, F.Cu at (102.6, 98.7)
- added C31: 10uF, Capacitor_SMD:C_0603_1608Metric, F.Cu at (127.3, 76.9)
- added C32: 10uF, Capacitor_SMD:C_0603_1608Metric, F.Cu at (127.3, 79.4)
- added C4: 22uF, Capacitor_SMD:C_1206_3216Metric, F.Cu at (88.2, 109.0)
- added D1: Green, LED_SMD:LED_0805_2012Metric, F.Cu at (127.5, 62.9)
- added D2: Red, LED_SMD:LED_0805_2012Metric, F.Cu at (127.5, 66.0)
- added J6: USB_C_Receptacle_USB2.0, Connector_USB:USB_C_Receptacle_HCTL_HC-TYPE-C-16P-01A, F.Cu at (125.7, 90.7)
- added L1: 3A+ 2.2uH, Inductor_SMD:L_SXN_SMDRI124, F.Cu at (143.8, 46.5)
- added L2: 3A+ 2.2uH, Inductor_SMD:L_SXN_SMDRI124, F.Cu at (107.0, 36.5)
- added L3: 3A+ 2.2uH, Inductor_SMD:L_SXN_SMDRI124, F.Cu at (92.6, 97.9)
- added R10: 220k, Resistor_SMD:R_0603_1608Metric, F.Cu at (107.4, 93.3)
- added R11: 22k, Resistor_SMD:R_0603_1608Metric, F.Cu at (107.4, 95.8)
- added R8: 220k, Resistor_SMD:R_0603_1608Metric, F.Cu at (107.4, 88.3)
- added R9: 30k, Resistor_SMD:R_0603_1608Metric, F.Cu at (107.4, 90.8)
- added U10: FUSB303BTMX, Package_DFN_QFN:Texas_X2QFN-12_1.6x1.6mm_P0.4mm, F.Cu at (121.8, 97.3)
- added U7: TPS563203, Package_TO_SOT_SMD:SOT-563, F.Cu at (111.3, 82.1)
- added U8: TLV76150DCYR, Package_TO_SOT_SMD:SOT-223-3_TabPin2, F.Cu at (110.3, 101.2)
- added U9: LP2985-3.3, Package_TO_SOT_SMD:SOT-23-5, F.Cu at (131.9, 78.0)
- C1: value 100nF -> 22uF; footprint Capacitor_SMD:C_0603_1608Metric -> Capacitor_SMD:C_1206_3216Metric
- C10, C12: value 100nF -> 10uF
- C6, C9: value 10uF -> 100nF
- U5: value MAX98306xDT -> TPS563203; footprint Package_DFN_QFN:TDFN-14-1EP_3x3mm_P0.4mm_EP1.78x2.35mm -> Package_TO_SOT_SMD:SOT-563
- moved U5 10.7 mm to (111.3, 78.7)
Connections:
- C1 pad 1: +5V -> /Battery charger/5VIn
- C10 pad 1: +3V3 -> Net-(U4-VNEG)
- C11 pad 1: +3.3VA -> Net-(U4-CAPP)
- C11 pad 2: GND -> Net-(U4-CAPM)
- C12 pad 1: +3.3VA -> Net-(U4-LDOO)
- C13 pad 1: +3.3VA -> Net-(U4-LDOO)
- C2 pad 1: Net-(C2-Pad1) -> /Battery charger/5VIn
- C2 pad 2: Net-(U3-BST) -> GND
- C5 pad 1: Net-(U4-VNEG) -> +3.3VA
- C6 pad 1: Net-(U4-LDOO) -> +3.3VA
- C7 pad 1: Net-(U4-LDOO) -> +3.3VA
- C8 pad 1: Net-(U4-CAPP) -> +3V3
- C8 pad 2: Net-(U4-CAPM) -> GND
- U3 pad 12: unconnected-(U3-TM-Pad12) -> Net-(U3-TM)
- U3 pad 16: +5V -> /Battery charger/5VIn
- U3 pad 2: +5V -> /Battery charger/5VIn
- U3 pad 5: Net-(C2-Pad1) -> Net-(C3-Pad1)
- U3 pad 6: Net-(C2-Pad1) -> Net-(C3-Pad1)
- U3 pad 9: unconnected-(U3-BAT-Pad9) -> +VBAT
- U5 pad 1: Net-(U5-PGND-Pad1) -> +VBAT
- U5 pad 2: unconnected-(U5-~{SHDN}-Pad2) -> Net-(U5-SW)
- U5 pad 3: unconnected-(U5-INL+-Pad3) -> GND
- U5 pad 4: unconnected-(U5-INL--Pad4) -> Net-(U5-BST)
- U5 pad 5: unconnected-(U5-GAIN-Pad5) -> +VBAT
- U5 pad 6: unconnected-(U5-INR--Pad6) -> Net-(U5-FB)
- U6 pad 1: unconnected-(U6-+OUT_L-Pad1) -> /Stereo amplifier/+OUT_L
- U6 pad 10: unconnected-(U6-INR-Pad10) -> Net-(U6-INR)
- U6 pad 11: unconnected-(U6-GND-Pad11) -> GND
- U6 pad 12: unconnected-(U6-~{SHND}-Pad12) -> +5VA
- U6 pad 13: unconnected-(U6-PVDDR-Pad13) -> +5VA
- U6 pad 14: unconnected-(U6--OUT_R-Pad14) -> /Stereo amplifier/-OUT_R
- U6 pad 15: unconnected-(U6-PGNDR-Pad15) -> GND
- U6 pad 16: unconnected-(U6-+OUT_R-Pad16) -> /Stereo amplifier/+OUT_R
- U6 pad 2: unconnected-(U6-PGNDL-Pad2) -> GND
- U6 pad 3: unconnected-(U6--OUT_L-Pad3) -> /Stereo amplifier/-OUT_L
- U6 pad 4: unconnected-(U6-PVDDL-Pad4) -> +5VA
- U6 pad 5: unconnected-(U6-~{MUTE}-Pad5) -> +5VA
- U6 pad 6: unconnected-(U6-VDD-Pad6) -> +5VA
- U6 pad 7: unconnected-(U6-INL-Pad7) -> Net-(U6-INL)
- U6 pad 8: unconnected-(U6-VREF-Pad8) -> Net-(U6-VREF)
- U6 pad 9: unconnected-(U6-MODE-Pad9) -> +5VA
